File: pcb/Win-split.kicad_sch (KiCad schematic)
At the start: 220 parts

Commit message: .
Parts:
- removed MC1: ~, Winkeebs:RP2040_ProMicro, symbol Winkeebs:RP2040_ProMicro
- removed MC2: ~, PCM_marbastlib-xp-promicroish:ProMicro_USBdn, symbol Winkeebs:RP2040_ProMicro
- added H1, H2, H3, H4: MountingHole, MountingHole:MountingHole_2.2mm_M2, symbol Mechanical:MountingHole
- added J1, J2: Conn_01x04_Socket, Connector_PinHeader_2.54mm:PinHeader_1x04_P2.54mm_Vertical, symbol Connector:Conn_01x04_Socket
- added S22, S31, S40: MX_stab, PCM_marbastlib-mx:STAB_MX_2u, symbol PCM_marbastlib-mx:MX_stab
- added S55, S64: MX_stab, PCM_marbastlib-mx:STAB_MX_2.25u, symbol PCM_marbastlib-mx:MX_stab
- added U1: RP2040_ProMicro, PCM_marbastlib-xp-promicroish:ProMicro_USBup, symbol Winkeebs:Arduino_ProMicro
- added U2: RP2040_ProMicro, PCM_marbastlib-xp-promicroish:ProMicro_USBdn, symbol Winkeebs:Arduino_ProMicro
- LED1, LED15, LED16, LED17, LED18, LED19, LED2, LED20, LED21, LED28, LED29, LED3, LED30, LED31, LED33, LED34, LED35, LED36, LED37, LED38, LED39, LED4, LED40, LED41, LED42, LED43, LED44, LED45, LED46, LED47, LED48, LED49, LED5, LED50, LED51, LED52, LED53, LED54, LED55, LED56, LED57, LED58, LED59, LED6, LED60, LED61, LED62, LED63, LED64, LED65, LED66, LED67, LED68, LED69, LED7, LED70: footprint PCM_marbastlib-mx:LED_MX_6028R -> PCM_marbastlib-mx:LED_MX_6028R-ROT
- MX16, MX61: footprint PCM_Switch_Keyboard_Hotswap_Kailh:SW_Hotswap_Kailh_MX_1.00u -> PCM_Switch_Keyboard_Hotswap_Kailh:SW_Hotswap_Kailh_MX_1.75u
- MX22, MX31, MX40: footprint PCM_Switch_Keyboard_Hotswap_Kailh:SW_Hotswap_Kailh_MX_1.00u -> PCM_Switch_Keyboard_Hotswap_Kailh:SW_Hotswap_Kailh_MX_2.00u
- MX28, MX29, MX30, MX65, MX66, MX67: footprint PCM_Switch_Keyboard_Hotswap_Kailh:SW_Hotswap_Kailh_MX_1.00u -> PCM_Switch_Keyboard_Hotswap_Kailh:SW_Hotswap_Kailh_MX_1.25u
- MX48, MX9: footprint PCM_Switch_Keyboard_Hotswap_Kailh:SW_Hotswap_Kailh_MX_1.00u -> PCM_Switch_Keyboard_Hotswap_Kailh:SW_Hotswap_Kailh_MX_1.50u
- MX55, MX64: footprint PCM_Switch_Keyboard_Hotswap_Kailh:SW_Hotswap_Kailh_MX_1.00u -> PCM_Switch_Keyboard_Hotswap_Kailh:SW_Hotswap_Kailh_MX_2.25u
- Reset1: footprint ScottoKeebs_Cutout:Cutout_MX_1.00u -> Button_Switch_SMD:SW_SPST_B3U-1000P; LCSC (none) -> C231329
- Reset2: footprint ScottoKeebs_Cutout:Cutout_MX_1.00u -> Button_Switch_SMD:SW_SPST_B3U-1000P
Connections:
- net ColL 0: now also U1.18 (GP28)
- net ColL 1: now also U1.19 (GP27)
- net ColL 2: now also U1.20 (GP26)
- net ColL 3: now also U1.21 (GP22)
- net ColL 4: now also U1.22 (GP20)
- net ColL 5: now also U1.23 (GP23)
- net ColL 6: now also U1.24 (GP21)
- net ColR 0: now also U2.17 (GP29)
- net ColR 1: now also U2.18 (GP28)
- net ColR 2: now also U2.19 (GP27)
- net ColR 3: now also U2.20 (GP26)
- net ColR 4: now also U2.21 (GP22)
- net ColR 5: now also MX46.1, MX54.1, MX61.1, MX68.1, U2.22 (GP20)
- net ColR 6: now also U2.23 (GP23)
- net ColR 7: now also U2.24 (GP21)
- net GND: now also Reset1.2, Reset2.2, J1.1 (Pin_1), J2.1 (Pin_1), U1.14 (GND), U1.3 (GND), U1.4 (GND), U2.12 (GP9), U2.14 (GND), U2.3 (GND), U2.4 (GND); no longer Reset1.1, Reset2.1
- net LED1: now also U1.2 (GP1-RX)
- net LED2: now also U2.2 (GP1-RX)
- net RAW2: now also U2.13 (RAW-5V); no longer LED33.1 (VDD), LED34.1 (VDD), LED35.1 (VDD), LED36.1 (VDD), LED37.1 (VDD), LED38.1 (VDD), LED39.1 (VDD), LED40.1 (VDD), LED41.1 (VDD), LED42.1 (VDD), LED43.1 (VDD), LED44.1 (VDD), LED45.1 (VDD), LED46.1 (VDD), LED47.1 (VDD), LED48.1 (VDD), LED49.1 (VDD), LED50.1 (VDD), LED51.1 (VDD), LED52.1 (VDD), LED53.1 (VDD), LED54.1 (VDD), LED55.1 (VDD), LED56.1 (VDD), LED57.1 (VDD), LED58.1 (VDD), LED59.1 (VDD), LED60.1 (VDD), LED61.1 (VDD), LED62.1 (VDD), LED63.1 (VDD), LED64.1 (VDD), LED65.1 (VDD), LED66.1 (VDD), LED67.1 (VDD), LED68.1 (VDD), LED69.1 (VDD), LED70.1 (VDD)
- net RowL 0: now also U1.7 (GP4)
- net RowL 1: now also U1.8 (GP5)
- net RowL 2: now also U1.9 (GP6)
- net RowL 3: now also U1.10 (GP7)
- net RowL 4: now also U1.11 (GP8)
- net RowR 0: now also U2.7 (GP4)
- net RowR 1: now also U2.8 (GP5)
- net RowR 2: now also U2.9 (GP6)
- net RowR 3: now also U2.10 (GP7)
- net RowR 4: now also U2.11 (GP8)
- net VCC: now also J1.2 (Pin_2), J2.2 (Pin_2), U1.12 (GP9), U1.16 (VCC-3V3), U2.16 (VCC-3V3)
- net SDA1: now reaches OLED1.4 (SDA)
- net SDA1: now also J1.4 (Pin_4), U1.5 (GP2)
- net SCL1: now reaches OLED1.3 (SCL)
- net SCL1: now also J1.3 (Pin_3), U1.6 (GP3)
- net at ESD1.4 (IO3): now also U1.1 (GP0-TX)
- net SDA2: now reaches OLED2.4 (SDA)
- net SDA2: now also J2.4 (Pin_4), U2.5 (GP2)
- net SCL2: now reaches OLED2.3 (SCL)
- net SCL2: now also J2.3 (Pin_3), U2.6 (GP3)
- net at ESD2.4 (IO3): now also U2.1 (GP0-TX)
- net RAW1 renamed +5V
- net +5V: now also LED33.1 (VDD), LED34.1 (VDD), LED35.1 (VDD), LED36.1 (VDD), LED37.1 (VDD), LED38.1 (VDD), LED39.1 (VDD), LED40.1 (VDD), LED41.1 (VDD), LED42.1 (VDD), LED43.1 (VDD), LED44.1 (VDD), LED45.1 (VDD), LED46.1 (VDD), LED47.1 (VDD), LED48.1 (VDD), LED49.1 (VDD), LED50.1 (VDD), LED51.1 (VDD), LED52.1 (VDD), LED53.1 (VDD), LED54.1 (VDD), LED55.1 (VDD), LED56.1 (VDD), LED57.1 (VDD), LED58.1 (VDD), LED59.1 (VDD), LED60.1 (VDD), LED61.1 (VDD), LED62.1 (VDD), LED63.1 (VDD), LED64.1 (VDD), LED65.1 (VDD), LED66.1 (VDD), LED67.1 (VDD), LED68.1 (VDD), LED69.1 (VDD), LED70.1 (VDD), U1.13 (RAW-5V)
- new net Reset1: Reset1.1, U1.15 (RST)
- new net Reset2: Reset2.1, U2.15 (RST)
- no-connect marks 31 -> 9
Other:
- note added: "Hand high"
- note added: "Hand low"
- moved on the sheet: OLED1, OLED2, Reset1, Reset2

Commit message: x
Parts:
- S22, S31, S40: footprint PCM_marbastlib-mx:STAB_MX_2u -> ScottoKeebs_Stabilizer:Stabilizer_MX_2.00u
- U1: footprint PCM_marbastlib-xp-promicroish:ProMicro_USBup -> winkeebs:RP2040_ProMicro_USBup; symbol Winkeebs:Arduino_ProMicro -> Winkeebs:RP2040_ProMicro; now in the parts list
- U2: footprint PCM_marbastlib-xp-promicroish:ProMicro_USBdn -> winkeebs:RP2040_ProMicro_USBdn; symbol Winkeebs:Arduino_ProMicro -> Winkeebs:RP2040_ProMicro; now in the parts list
Connections:
- net +5V: now also U1.5v; no longer U1.13 (RAW-5V)
- net ColL 0: now also U1.28; no longer U1.18 (GP28)
- net ColL 1: now also U1.27; no longer U1.19 (GP27)
- net ColL 2: now also U1.26; no longer U1.20 (GP26)
- net ColL 3: now also U1.22; no longer U1.21 (GP22)
- net ColL 4: now also U1.20; no longer U1.22 (GP20)
- net ColL 6: now also U1.21; no longer U1.24 (GP21)
- net ColR 0: now also U2.29; no longer U2.17 (GP29)
- net ColR 1: now also U2.28; no longer U2.18 (GP28)
- net ColR 2: now also U2.27; no longer U2.19 (GP27)
- net ColR 3: now also U2.26; no longer U2.20 (GP26)
- net ColR 4: now also U2.22; no longer U2.21 (GP22)
- net ColR 5: now also U2.20; no longer U2.22 (GP20)
- net ColR 7: now also U2.21; no longer U2.24 (GP21)
- net GND: now also U1.G (GND), U2.9, U2.G (GND); no longer U1.14 (GND), U1.3 (GND), U1.4 (GND), U2.12 (GP9), U2.14 (GND), U2.3 (GND), U2.4 (GND)
- net LED1: now also U1.1 (RX); no longer U1.2 (GP1-RX)
- net LED2: now also U2.1 (RX); no longer U2.2 (GP1-RX)
- net RAW2: now also U2.5v; no longer U2.13 (RAW-5V)
- net Reset1: now also U1.RST; no longer U1.15 (RST)
- net Reset2: now also U2.RST; no longer U2.15 (RST)
- net RowL 0: now also U1.4; no longer U1.7 (GP4)
- net RowL 1: now also U1.5; no longer U1.8 (GP5)
- net RowL 2: now also U1.6; no longer U1.9 (GP6)
- net RowL 3: now also U1.7; no longer U1.10 (GP7)
- net RowL 4: now also U1.8; no longer U1.11 (GP8)
- net RowR 0: now also U2.4; no longer U2.7 (GP4)
- net RowR 1: now also U2.5; no longer U2.8 (GP5)
- net RowR 2: now also U2.6; no longer U2.9 (GP6)
- net RowR 3: now also U2.7; no longer U2.10 (GP7)
- net RowR 4: now also U2.8; no longer U2.11 (GP8)
- net SCL1: now also U1.3 (SCL); no longer U1.6 (GP3)
- net SCL2: now also U2.3 (SCL); no longer U2.6 (GP3)
- net SDA1: now also U1.2 (SDA); no longer U1.5 (GP2)
- net SDA2: now also U2.2 (SDA); no longer U2.5 (GP2)
- net VCC: now also U1.3v3, U1.9, U2.3v3; no longer U1.12 (GP9), U1.16 (VCC-3V3), U2.16 (VCC-3V3)
- net at ESD1.4 (IO3): now also U1.0 (TX); no longer U1.1 (GP0-TX)
- net at ESD2.4 (IO3): now also U2.0 (TX); no longer U2.1 (GP0-TX)
- no-connect marks 9 -> 17
Changed lines of the file:
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@@
   )
   (no_connect (at 55.88 44.45))
+  (no_connect (at 125.73 39.37))
+  (no_connect (at 107.95 41.91))
   (no_connect (at 81.28 39.37))
   (no_connect (at 133.35 54.61))
+  (no_connect (at 128.27 76.2))
+  (no_connect (at 133.35 41.91))
   (no_connect (at 727.71 48.26))
+  (no_connect (at 113.03 76.2))
+  (no_connect (at 125.73 76.2))
   (no_connect (at 350.52 317.5))
   (no_connect (at 702.31 53.34))
+  (no_connect (at 123.19 76.2))
   (no_connect (at 40.64 41.91))
   (no_connect (at 687.07 50.8))
+  (no_connect (at 115.57 39.37))
   (no_connect (at 604.52 317.5))
   (wire (pts (xy 571.5 248.92) (xy 571.5 254))
@@
       (effects (font (size 1.27 1.27)) (justify left))
     )
-    (property "Footprint" "PCM_marbastlib-mx:STAB_MX_2u" (at 717.55 114.3 0)
+    (property "Footprint" "ScottoKeebs_Stabilizer:Stabilizer_MX_2.00u" (at 717.55 114.3 0)
       (effects (font (size 1.27 1.27)) hide)
     )
@@
       (effects (font (size 1.27 1.27)) (justify left))
     )
-    (property "Footprint" "PCM_marbastlib-mx:STAB_MX_2u" (at 67.31 158.75 0)
+    (property "Footprint" "ScottoKeebs_Stabilizer:Stabilizer_MX_2.00u" (at 67.31 158.75 0)
       (effects (font (size 1.27 1.27)) hide)
     )
@@
     )
   )
-  (symbol (lib_id "Winkeebs:Arduino_ProMicro") (at 120.65 58.42 0) (unit 1)
-    (in_bom no) (on_board yes) (dnp no) (fields_autoplaced)
-    (property "Reference" "U1" (at 120.65 36.83 0)
-      (effects (font (size 1.27 1.27)))
+  (symbol (lib_id "Winkeebs:RP2040_ProMicro") (at 120.65 58.42 0) (unit 1)
+    (in_bom yes) (on_board yes) (dnp no) (fields_autoplaced)
+    (property "Reference" "U1" (at 127.3811 33.02 0)
+      (effects (font (size 1.27 1.27)) (justify left))
     )
-    (property "Value" "RP2040_ProMicro" (at 120.65 39.37 0)
-      (effects (font (size 1.27 1.27)))
+    (property "Value" "RP2040_ProMicro" (at 127.3811 35.56 0)
+      (effects (font (size 1.27 1.27)) (justify left))
     )
-    (property "Footprint" "PCM_marbastlib-xp-promicroish:ProMicro_USBup" (at 120.65 88.9 0)
+    (property "Footprint" "winkeebs:RP2040_ProMicro_USBup" (at 120.65 27.94 0)
       (effects (font (size 1.27 1.27)) hide)
     )
-    (property "Datasheet" "" (at 107.95 44.45 0)
+    (property "Datasheet" "" (at 120.65 38.1 0)
       (effects (font (size 1.27 1.27)) hide)
     )
@@
     (pin "3")
     (pin "21")
-    (pin "17")
+    (pin "0")
     (pin "11")
     (pin "12")
@@
     (pin "20")
     (pin "2")
-    (pin "19")
+    (pin "5v")
     (pin "18")
     (pin "1")
@@
     (pin "14")
     (pin "24")
+    (pin "BOOT")
+    (pin "G")
+    (pin "G")
+    (pin "G")
+    (pin "RST")
+    (pin "25")
+    (pin "26")
+    (pin "27")
+    (pin "28")
+    (pin "29")
+    (pin "3v3")
     (instances
       (project "Win-split"
@@
       (effects (font (size 1.27 1.27)) (justify left))
     )
-    (property "Footprint" "PCM_marbastlib-mx:STAB_MX_2u" (at 67.31 168.91 0)
+    (property "Footprint" "ScottoKeebs_Stabilizer:Stabilizer_MX_2.00u" (at 67.31 168.91 0)
       (effects (font (size 1.27 1.27)) hide)
     )
@@
     )
   )
-  (symbol (lib_id "Winkeebs:Arduino_ProMicro") (at 767.08 67.31 0) (unit 1)
-    (in_bom no) (on_board yes) (dnp no) (fields_autoplaced)
-    (property "Reference" "U2" (at 767.08 45.72 0)
-      (effects (font (size 1.27 1.27)))
+  (symbol (lib_id "Winkeebs:RP2040_ProMicro") (at 767.08 67.31 0) (unit 1)
+    (in_bom yes) (on_board yes) (dnp no) (fields_autoplaced)
+    (property "Reference" "U2" (at 773.8111 41.91 0)
+      (effects (font (size 1.27 1.27)) (justify left))
     )
-    (property "Value" "RP2040_ProMicro" (at 767.08 48.26 0)
-      (effects (font (size 1.27 1.27)))
+    (property "Value" "RP2040_ProMicro" (at 773.8111 44.45 0)
+      (effects (font (size 1.27 1.27)) (justify left))
     )
-    (property "Footprint" "PCM_marbastlib-xp-promicroish:ProMicro_USBdn" (at 767.08 97.79 0)
+    (property "Footprint" "winkeebs:RP2040_ProMicro_USBdn" (at 767.08 36.83 0)
       (effects (font (size 1.27 1.27)) hide)
     )
-    (property "Datasheet" "" (at 754.38 53.34 0)
+    (property "Datasheet" "" (at 767.08 46.99 0)
       (effects (font (size 1.27 1.27)) hide)
     )
@@
     (pin "18")
     (pin "2")
-    (pin "19")
+    (pin "0")
     (pin "6")
     (pin "15")
-    (pin "17")
+    (pin "25")
     (pin "12")
     (pin "11")
@@
     (pin "4")
     (pin "1")
+    (pin "26")
+    (pin "27")
+    (pin "28")
+    (pin "29")
+    (pin "3v3")
+    (pin "5v")
+    (pin "BOOT")
+    (pin "G")
+    (pin "G")
+    (pin "G")
+    (pin "RST")
     (instances
       (project "Win-split"
