File: pcb/_autosave-Win-split.kicad_pcb (KiCad board)
At the start: 2 copper layers, 4.1 x 3.8 mm, 235 parts, among them J1 Conn_01x04_Socket, J2 Conn_01x04_Socket, SW1 ROT_SKYLOONG_HS, U1 RP2040_ProMicro, U2 RP2040_ProMicro

Commit message: x
Parts:
- removed D71: Diode, ScottoKeebs_Components:Diode_SOD-123
- removed LED71: MX_SK6812MINI-E, PCM_marbastlib-mx:LED_MX_6028R-ROT
- removed MX71: MX_SW_HS, ScottoKeebs_Hotswap:Hotswap_MX_1.25u
- removed SW1: ROT_SKYLOONG_HS, PCM_marbastlib-various:ROT_SKYLOONG_HS-Switch
- MX1, MX10, MX11, MX12, MX13, MX14, MX15, MX17, MX18, MX19, MX2, MX20, MX21, MX23, MX24, MX25, MX26, MX27, MX3, MX32, MX33, MX34, MX35, MX36, MX37, MX38, MX39, MX4, MX41, MX42, MX43, MX44, MX45, MX46, MX47, MX49, MX5, MX50, MX51, MX52, MX53, MX54, MX56, MX57, MX58, MX59, MX6, MX60, MX62, MX63, MX68, MX69, MX7, MX70, MX8: footprint ScottoKeebs_Hotswap:Hotswap_MX_1.00u -> PCM_Switch_Keyboard_Hotswap_Kailh:SW_Hotswap_Kailh_MX_1.00u
- MX16, MX61: footprint ScottoKeebs_Hotswap:Hotswap_MX_1.75u -> PCM_Switch_Keyboard_Hotswap_Kailh:SW_Hotswap_Kailh_MX_1.75u
- MX22, MX31, MX40: footprint ScottoKeebs_Hotswap:Hotswap_MX_2.00u -> PCM_Switch_Keyboard_Hotswap_Kailh:SW_Hotswap_Kailh_MX_2.00u
- MX28, MX29, MX30, MX65, MX66, MX67: footprint ScottoKeebs_Hotswap:Hotswap_MX_1.25u -> PCM_Switch_Keyboard_Hotswap_Kailh:SW_Hotswap_Kailh_MX_1.25u
- MX48, MX9: footprint ScottoKeebs_Hotswap:Hotswap_MX_1.50u -> PCM_Switch_Keyboard_Hotswap_Kailh:SW_Hotswap_Kailh_MX_1.50u
- MX55, MX64: footprint ScottoKeebs_Hotswap:Hotswap_MX_2.25u -> PCM_Switch_Keyboard_Hotswap_Kailh:SW_Hotswap_Kailh_MX_2.25u
- S22, S31, S40: footprint PCM_marbastlib-mx:STAB_MX_2u -> ScottoKeebs_Stabilizer:Stabilizer_MX_2.00u
Connections:
- D15 pad 2: unconnected-(D15-A-Pad2) -> Net-(D15-A)
- MX15 pad 1: unconnected-(MX15-Pad1) -> ColL 0
- MX15 pad 2: ColL 0 -> Net-(D15-A)
Routing:
- net ColL 0: track 79.3 -> 74.9 mm
- net Net-(D15-A): track 0.00 -> 4.39 mm
Other:
- board size 4.1 x 3.8 mm -> 402.1 x 120.7 mm
