File: pcb/Win-split-before-led_swap.kicad_sch (KiCad schematic)
At the start: 242 parts, among them J1 Conn_01x04_Socket, J2 Conn_01x04_Socket, SW1 ROT_SKYLOONG_HS, SW2 ROT_SKYLOONG_HS, U1 RP2040_ProMicro, U2 RP2040_ProMicro

Commit message: pre-del button
Parts:
- removed SW1, SW2: ROT_SKYLOONG_HS, PCM_marbastlib-various:ROT_SKYLOONG_HS-Switch, symbol PCM_marbastlib-various:ROT_SKYLOONG_HS-Switch
- H1, H10, H2, H3, H4, H5, H6, H7, H8, H9: footprint winkeebs:HOLE_M2 -> winkeebs:HOLE_M2_TH
Connections:
- net ROTA: no longer names the net of U1.14
- net ROTB: no longer names the net of U1.13
- net ROTS: no longer names the net of U1.12
- no-connect marks 28 -> 17
