File: pcb/Win-split.kicad_pcb (KiCad board)
At the start: 2 copper layers, 14 x 14 mm, 220 parts

Commit message: .
Parts:
- removed ESDL1, ESDR1: SRV05-4, PCM_marbastlib-various:SOT-23-6-routable
- removed MCUL1, MCUR1: ~, PCM_marbastlib-xp-promicroish:ProMicro_USBdn
- removed OLEDL1, OLEDR1: OLED_128x32, ScottoKeebs_Components:OLED_128x32
- removed ResetL1, ResetR1: Switch, ScottoKeebs_Cutout:Cutout_MX_1.00u
- removed TRRSL1, TRRSR1: PJ-320A, Keebio:TRRS-PJ-320A
- added ESD1: SRV05-4, PCM_marbastlib-various:SOT-23-6-routable, F.Cu at (238.4, 140.0)
- added ESD2: SRV05-4, PCM_marbastlib-various:SOT-23-6-routable, F.Cu at (261.6, 140.2)
- added H1: MountingHole, MountingHole:MountingHole_2.2mm_M2, F.Cu at (257.3, 375.4)
- added H2: MountingHole, MountingHole:MountingHole_2.2mm_M2, F.Cu at (257.3, 381.3)
- added H3: MountingHole, MountingHole:MountingHole_2.2mm_M2, F.Cu at (257.3, 387.3)
- added H4: MountingHole, MountingHole:MountingHole_2.2mm_M2, F.Cu at (257.3, 393.2)
- added J1: Conn_01x04_Socket, Connector_PinHeader_2.54mm:PinHeader_1x04_P2.54mm_Vertical, F.Cu at (227.6, 156.5)
- added J2: Conn_01x04_Socket, Connector_PinHeader_2.54mm:PinHeader_1x04_P2.54mm_Vertical, F.Cu at (280.2, 156.5)
- added OLED1: OLED_128x32, ScottoKeebs_Components:OLED_128x32, F.Cu at (217.8, 158.1)
- added OLED2: OLED_128x32, ScottoKeebs_Components:OLED_128x32, F.Cu at (270.4, 158.1)
- added Reset1: Switch, Button_Switch_SMD:SW_SPST_B3U-1000P, F.Cu at (238.4, 148.3)
- added Reset2: Switch, Button_Switch_SMD:SW_SPST_B3U-1000P, F.Cu at (261.6, 148.5)
- added S22: MX_stab, PCM_marbastlib-mx:STAB_MX_2u, F.Cu at (96.8, 192.3)
- added S31: MX_stab, PCM_marbastlib-mx:STAB_MX_2u, F.Cu at (212.3, 202.6)
- added S40: MX_stab, PCM_marbastlib-mx:STAB_MX_2u, F.Cu at (440.1, 142.6)
- added S55: MX_stab, PCM_marbastlib-mx:STAB_MX_2.25u, F.Cu at (424.0, 177.8)
- added S64: MX_stab, PCM_marbastlib-mx:STAB_MX_2.25u, F.Cu at (290.1, 202.6)
- added TRRS1: TRRS, ScottoKeebs_Components:TRRS_PJ-320A, F.Cu at (238.4, 121.4)
- added TRRS2: TRRS, ScottoKeebs_Components:TRRS_PJ-320A, F.Cu at (261.6, 121.4)
- added U1: RP2040_ProMicro, PCM_marbastlib-xp-promicroish:ProMicro_USBup, F.Cu at (223.7, 137.1)
- added U2: RP2040_ProMicro, PCM_marbastlib-xp-promicroish:ProMicro_USBdn, F.Cu at (276.3, 137.1)
- LED1, LED15, LED16, LED17, LED18, LED19, LED2, LED20, LED21, LED28, LED29, LED3, LED30, LED31, LED33, LED34, LED35, LED36, LED37, LED38, LED39, LED4, LED40, LED41, LED42, LED43, LED44, LED45, LED46, LED47, LED48, LED49, LED5, LED50, LED51, LED52, LED53, LED54, LED55, LED56, LED57, LED58, LED59, LED6, LED60, LED61, LED62, LED63, LED64, LED65, LED66, LED67, LED68, LED69, LED7, LED70: footprint PCM_marbastlib-mx:LED_MX_6028R -> PCM_marbastlib-mx:LED_MX_6028R-ROT
- MX1, MX10, MX11, MX12, MX13, MX14, MX15, MX17, MX18, MX19, MX2, MX20, MX21, MX23, MX24, MX25, MX26, MX27, MX3, MX32, MX33, MX34, MX35, MX36, MX37, MX38, MX39, MX4, MX41, MX42, MX43, MX44, MX45, MX46, MX47, MX49, MX5, MX50, MX51, MX52, MX53, MX54, MX56, MX57, MX58, MX59, MX6, MX60, MX62, MX63, MX68, MX69, MX7, MX70, MX8: footprint ScottoKeebs_Hotswap:Hotswap_MX_1.00u -> PCM_Switch_Keyboard_Hotswap_Kailh:SW_Hotswap_Kailh_MX_1.00u
- MX16, MX61: footprint ScottoKeebs_Hotswap:Hotswap_MX_1.00u -> PCM_Switch_Keyboard_Hotswap_Kailh:SW_Hotswap_Kailh_MX_1.75u
- MX22, MX31, MX40: footprint ScottoKeebs_Hotswap:Hotswap_MX_1.00u -> PCM_Switch_Keyboard_Hotswap_Kailh:SW_Hotswap_Kailh_MX_2.00u
- MX28, MX29, MX30, MX65, MX66, MX67: footprint ScottoKeebs_Hotswap:Hotswap_MX_1.00u -> PCM_Switch_Keyboard_Hotswap_Kailh:SW_Hotswap_Kailh_MX_1.25u
- MX48, MX9: footprint ScottoKeebs_Hotswap:Hotswap_MX_1.00u -> PCM_Switch_Keyboard_Hotswap_Kailh:SW_Hotswap_Kailh_MX_1.50u
- MX55, MX64: footprint ScottoKeebs_Hotswap:Hotswap_MX_1.00u -> PCM_Switch_Keyboard_Hotswap_Kailh:SW_Hotswap_Kailh_MX_2.25u
- moved LED15 108.1 mm to (70.3, 184.5), turned to -166 degrees
- moved MX15 107.9 mm to (69.1, 179.6), turned to 14 degrees
- moved LED8 106.1 mm to (70.3, 164.9), turned to -166 degrees
- moved MX8 105.9 mm to (69.1, 159.9), turned to 14 degrees
- moved LED28 104.4 mm to (105.0, 215.1), turned to -166 degrees
- moved LED1 104.2 mm to (70.4, 145.2), turned to -166 degrees
- moved MX1 104.1 mm to (69.1, 140.3), turned to 14 degrees
- moved MX28 104.0 mm to (103.7, 210.2), turned to 14 degrees
- moved MX40 103.8 mm to (440.1, 142.6), turned to -14 degrees
- moved LED22 103.6 mm to (98.0, 197.2), turned to -166 degrees
- moved LED40 103.6 mm to (438.9, 147.5), turned to 166 degrees
- moved MX22 103.3 mm to (96.8, 192.3), turned to 14 degrees
- moved MX48 102.7 mm to (435.5, 161.1), turned to -14 degrees
- moved LED70 102.6 mm to (438.9, 226.1), turned to 166 degrees
- moved LED48 102.6 mm to (434.3, 166.0), turned to 166 degrees
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Connections:
- net Hand renamed GND
- LED1 pad 1: RAWL -> +5V
- LED1 pad 3: LEDL -> LED1
- LED10 pad 1: RAWL -> +5V
- LED11 pad 1: RAWL -> +5V
- LED12 pad 1: RAWL -> +5V
- LED13 pad 1: RAWL -> +5V
- LED13 pad 2: Net-(LED13-DOUT) -> Net-(LED12-DIN)
- LED14 pad 1: RAWL -> +5V
- LED14 pad 2: Net-(LED14-DOUT) -> Net-(LED13-DIN)
- LED14 pad 3: Net-(LED13-DOUT) -> Net-(LED14-DIN)
- LED15 pad 1: RAWL -> +5V
- LED15 pad 3: Net-(LED14-DOUT) -> Net-(LED15-DIN)
- LED16 pad 1: RAWL -> +5V
- LED17 pad 1: RAWL -> +5V
- LED18 pad 1: RAWL -> +5V
- LED19 pad 1: RAWL -> +5V
- LED19 pad 2: unconnected-(LED19-DOUT-Pad2) -> Net-(LED19-DOUT)
- LED19 pad 3: Net-(LED19-DIN) -> Net-(LED18-DOUT)
- LED2 pad 1: RAWL -> +5V
- LED20 pad 1: unconnected-(LED20-VDD-Pad1) -> +5V
- LED20 pad 2: Net-(LED19-DIN) -> Net-(LED20-DOUT)
- LED20 pad 3: Net-(LED20-DIN) -> Net-(LED19-DOUT)
- LED21 pad 1: RAWL -> +5V
- LED21 pad 2: Net-(LED20-DIN) -> Net-(LED21-DOUT)
- LED21 pad 3: Net-(LED21-DIN) -> Net-(LED20-DOUT)
- LED22 pad 1: RAWL -> +5V
- LED22 pad 2: Net-(LED21-DIN) -> Net-(LED22-DOUT)
- LED23 pad 1: RAWL -> +5V
- LED24 pad 1: RAWL -> +5V
- LED25 pad 1: RAWL -> +5V
- LED25 pad 2: Net-(LED25-DOUT) -> Net-(LED24-DIN)
- LED25 pad 3: unconnected-(LED25-DIN-Pad3) -> Net-(LED25-DIN)
- LED26 pad 1: RAWL -> +5V
- LED26 pad 2: Net-(LED26-DOUT) -> Net-(LED25-DIN)
- LED26 pad 3: Net-(LED25-DOUT) -> Net-(LED26-DIN)
- LED27 pad 1: RAWL -> +5V
- LED27 pad 2: Net-(LED27-DOUT) -> Net-(LED26-DIN)
- LED27 pad 3: Net-(LED26-DOUT) -> Net-(LED21-DOUT)
- LED28 pad 1: RAWL -> +5V
- LED28 pad 3: Net-(LED27-DOUT) -> Net-(LED22-DOUT)
- LED29 pad 1: RAWL -> +5V
- LED29 pad 2: unconnected-(LED29-DOUT-Pad2) -> Net-(LED29-DOUT)
- LED3 pad 1: RAWL -> +5V
- LED30 pad 1: RAWR -> +5V
- LED30 pad 3: LEDR -> Net-(LED29-DOUT)
- LED31 pad 1: RAWR -> +5V
- LED32 pad 1: RAWR -> +5V
- LED32 pad 2: Net-(LED32-DOUT) -> unconnected-(LED32-DOUT-Pad2)
- LED33 pad 1: RAWR -> +5V
- LED33 pad 3: Net-(LED32-DOUT) -> LED2
- LED34 pad 1: RAWR -> +5V
- LED35 pad 1: RAWR -> +5V
- LED36 pad 1: RAWR -> +5V
- LED37 pad 1: RAWR -> +5V
- LED38 pad 1: RAWR -> +5V
- LED39 pad 1: RAWR -> +5V
- LED39 pad 3: Net-(LED39-DIN) -> Net-(LED38-DOUT)
- LED4 pad 1: RAWL -> +5V
- LED40 pad 1: RAWR -> +5V
- LED40 pad 2: Net-(LED39-DIN) -> Net-(LED40-DOUT)
- LED40 pad 3: Net-(LED40-DIN) -> Net-(LED39-DOUT)
- LED41 pad 1: RAWR -> +5V
- LED41 pad 2: Net-(LED40-DIN) -> Net-(LED41-DOUT)
- LED42 pad 1: RAWR -> +5V
- LED43 pad 1: RAWR -> +5V
- LED44 pad 1: RAWR -> +5V
- LED45 pad 1: RAWR -> +5V
- LED46 pad 1: RAWR -> +5V
- LED47 pad 1: RAWR -> +5V
- LED47 pad 3: Net-(LED38-DOUT) -> Net-(LED47-DIN)
- LED48 pad 1: RAWR -> +5V
- LED48 pad 2: Net-(LED48-DOUT) -> Net-(LED47-DIN)
- LED48 pad 3: Net-(LED39-DOUT) -> Net-(LED40-DOUT)
- LED49 pad 1: RAWR -> +5V
- LED49 pad 3: Net-(LED48-DOUT) -> Net-(LED41-DOUT)
- LED5 pad 1: RAWL -> +5V
- LED5 pad 2: unconnected-(LED5-DOUT-Pad2) -> Net-(LED5-DOUT)
- LED50 pad 1: RAWR -> +5V
- LED51 pad 1: RAWR -> +5V
- LED52 pad 1: RAWR -> +5V
- LED53 pad 1: RAWR -> +5V
- LED54 pad 1: RAWR -> +5V
- LED55 pad 1: RAWR -> +5V
- LED56 pad 1: RAWR -> +5V
- LED56 pad 3: Net-(LED55-DOUT) -> Net-(LED56-DIN)
- LED57 pad 1: RAWL -> +5V
- LED57 pad 2: Net-(LED24-DIN) -> Net-(LED56-DIN)
- LED57 pad 3: Net-(LED18-DOUT) -> Net-(LED57-DIN)
- LED58 pad 1: RAWR -> +5V
- LED58 pad 2: Net-(LED58-DOUT) -> Net-(LED57-DIN)
- LED59 pad 1: RAWR -> +5V
- LED6 pad 1: RAWL -> +5V
- LED6 pad 2: Net-(LED12-DIN) -> Net-(LED6-DOUT)
- LED6 pad 3: unconnected-(LED6-DIN-Pad3) -> Net-(LED5-DOUT)
- LED60 pad 1: RAWR -> +5V
- LED61 pad 1: RAWR -> +5V
- LED62 pad 1: RAWR -> +5V
- LED62 pad 3: Net-(LED62-DIN) -> Net-(LED55-DOUT)
- LED63 pad 1: RAWR -> +5V
- LED63 pad 2: Net-(LED62-DIN) -> Net-(LED63-DOUT)
- LED63 pad 3: Net-(LED63-DIN) -> Net-(LED56-DOUT)
- LED64 pad 1: RAWR -> +5V
- LED64 pad 2: Net-(LED63-DIN) -> Net-(LED64-DOUT)
- LED64 pad 3: Net-(LED56-DOUT) -> Net-(LED63-DOUT)
- LED65 pad 1: RAWR -> +5V
- LED65 pad 3: Net-(LED58-DOUT) -> Net-(LED64-DOUT)
- LED66 pad 1: RAWR -> +5V
- LED67 pad 1: RAWR -> +5V
- LED68 pad 1: RAWR -> +5V
- LED69 pad 1: RAWR -> +5V
- LED7 pad 1: RAWL -> +5V
- LED7 pad 2: Net-(LED13-DIN) -> Net-(LED14-DIN)
- LED7 pad 3: Net-(LED7-DIN) -> Net-(LED6-DOUT)
- LED70 pad 1: RAWR -> +5V
- LED8 pad 1: RAWL -> +5V
- LED8 pad 2: Net-(LED7-DIN) -> Net-(LED15-DIN)
- LED9 pad 1: RAWL -> +5V
Routing:
- net RowR 4: track 0.00 -> 191.4 mm, vias 0 -> 14
- net RowR 0: track 0.00 -> 172.3 mm, vias 0 -> 15
- net RowL 4: track 0.00 -> 171.0 mm, vias 0 -> 8
- net RowR 1: track 0.00 -> 167.0 mm, vias 0 -> 16
- net RowR 3: track 0.00 -> 156.7 mm, vias 0 -> 14
- net RowR 2: track 0.00 -> 154.3 mm, vias 0 -> 14
- net RowL 2: track 0.00 -> 152.4 mm, vias 0 -> 12
- net RowL 1: track 0.00 -> 145.2 mm, vias 0 -> 12
- net RowL 0: track 0.00 -> 144.6 mm, vias 0 -> 9
- net RowL 3: track 0.00 -> 142.0 mm, vias 0 -> 10
- net ColL 6: track 0.00 -> 118.9 mm, vias 0 -> 3
- net ColR 1: track 0.00 -> 102.2 mm, vias 0 -> 2
- net ColL 5: track 0.00 -> 101.3 mm, vias 0 -> 2
- net ColL 1: track 0.00 -> 100.2 mm, vias 0 -> 1
- net ColL 4: track 0.00 -> 99.6 mm, vias 0 -> 1
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Other:
- board size 14 x 14 mm -> 4.1 x 3.8 mm

Commit message: pre-del button
Parts:
- removed S31, S40: MX_stab, PCM_marbastlib-mx:STAB_MX_2u
- removed S55, S64: MX_stab, PCM_marbastlib-mx:STAB_MX_2.25u
- added D71: Diode, ScottoKeebs_Components:Diode_SOD-123, B.Cu at (447.6, 138.2)
- added H10: MountingHole_Pad, winkeebs:HOLE_M2, F.Cu at (432.5, 125.0)
- added H5: MountingHole_Pad, winkeebs:HOLE_M2, F.Cu at (65.2, 125.0)
- added H6: MountingHole_Pad, winkeebs:HOLE_M2, F.Cu at (306.6, 48.8)
- added H7: MountingHole_Pad, winkeebs:HOLE_M2, F.Cu at (419.5, 61.8)
- added H8: MountingHole_Pad, winkeebs:HOLE_M2, F.Cu at (307.2, 107.2)
- added H9: MountingHole_Pad, winkeebs:HOLE_M2, F.Cu at (363.2, 107.7)
- added LED71: MX_SK6812MINI-E, winkeebs:LED_MX_6028R-ROT, B.Cu at (438.2, 141.5)
- added MX71: MX_SW_HS, ScottoKeebs_Hotswap:Hotswap_MX_1.00u, F.Cu at (439.4, 136.5)
- added S32: MX_stab, ScottoKeebs_Stabilizer:Stabilizer_MX_2.00u, F.Cu at (210.7, 118.0)
- added S41: MX_stab, ScottoKeebs_Stabilizer:Stabilizer_MX_2.00u, F.Cu at (439.4, 58.0)
- added S56: MX_stab, ScottoKeebs_Stabilizer:Stabilizer_MX_2.00u, F.Cu at (423.2, 93.2)
- added S65: MX_stab, ScottoKeebs_Stabilizer:Stabilizer_MX_2.00u, F.Cu at (289.3, 118.0)
- added SW1: ROT_SKYLOONG_HS, PCM_marbastlib-various:ROT_SKYLOONG_HS-Switch, F.Cu at (49.1, 60.3)
- added SW2: ROT_SKYLOONG_HS, PCM_marbastlib-various:ROT_SKYLOONG_HS-Switch, F.Cu at (58.3, 136.5)
- H1, H2, H3, H4: value MountingHole -> MountingHole_Pad; footprint MountingHole:MountingHole_2.2mm_M2 -> winkeebs:HOLE_M2
- LED1, LED15, LED16, LED17, LED18, LED19, LED2, LED20, LED21, LED28, LED29, LED3, LED30, LED31, LED33, LED34, LED35, LED36, LED37, LED38, LED39, LED4, LED40, LED41, LED5, LED50, LED51, LED52, LED53, LED54, LED55, LED56, LED6, LED64, LED65, LED66, LED67, LED68, LED69, LED7, LED70: footprint PCM_marbastlib-mx:LED_MX_6028R-ROT -> winkeebs:LED_MX_6028R-ROT
- LED10, LED11, LED12, LED13, LED14, LED22, LED23, LED24, LED25, LED26, LED27, LED8, LED9: footprint PCM_marbastlib-mx:LED_MX_6028R -> winkeebs:LED_MX_6028R
- LED32: footprint PCM_marbastlib-mx:LED_MX_6028R -> winkeebs:LED_MX_6028R-ROT
- LED42, LED43, LED44, LED45, LED46, LED47, LED48, LED49, LED57, LED58, LED59, LED60, LED61, LED62, LED63: footprint PCM_marbastlib-mx:LED_MX_6028R-ROT -> winkeebs:LED_MX_6028R
- MX1, MX10, MX11, MX12, MX13, MX14, MX15, MX17, MX18, MX19, MX2, MX20, MX21, MX23, MX24, MX25, MX26, MX27, MX3, MX33, MX34, MX35, MX36, MX37, MX38, MX39, MX4, MX42, MX43, MX44, MX45, MX46, MX47, MX5, MX50, MX51, MX52, MX53, MX54, MX57, MX58, MX59, MX6, MX60, MX63, MX69, MX7, MX70, MX8: footprint PCM_Switch_Keyboard_Hotswap_Kailh:SW_Hotswap_Kailh_MX_1.00u -> ScottoKeebs_Hotswap:Hotswap_MX_1.00u
- MX16: footprint PCM_Switch_Keyboard_Hotswap_Kailh:SW_Hotswap_Kailh_MX_1.75u -> ScottoKeebs_Hotswap:Hotswap_MX_1.75u
- MX22: footprint PCM_Switch_Keyboard_Hotswap_Kailh:SW_Hotswap_Kailh_MX_2.00u -> ScottoKeebs_Hotswap:Hotswap_MX_2.00u
- MX28: footprint PCM_Switch_Keyboard_Hotswap_Kailh:SW_Hotswap_Kailh_MX_1.25u -> ScottoKeebs_Hotswap:Hotswap_MX_1.00u
- MX29, MX30, MX66, MX67: footprint PCM_Switch_Keyboard_Hotswap_Kailh:SW_Hotswap_Kailh_MX_1.25u -> ScottoKeebs_Hotswap:Hotswap_MX_1.25u
- MX31: footprint PCM_Switch_Keyboard_Hotswap_Kailh:SW_Hotswap_Kailh_MX_2.00u -> ScottoKeebs_Hotswap:Hotswap_MX_1.25u
- MX32, MX41: footprint PCM_Switch_Keyboard_Hotswap_Kailh:SW_Hotswap_Kailh_MX_1.00u -> ScottoKeebs_Hotswap:Hotswap_MX_2.00u
- MX40: footprint PCM_Switch_Keyboard_Hotswap_Kailh:SW_Hotswap_Kailh_MX_2.00u -> ScottoKeebs_Hotswap:Hotswap_MX_1.00u
- MX48: footprint PCM_Switch_Keyboard_Hotswap_Kailh:SW_Hotswap_Kailh_MX_1.50u -> ScottoKeebs_Hotswap:Hotswap_MX_1.00u
- MX49: footprint PCM_Switch_Keyboard_Hotswap_Kailh:SW_Hotswap_Kailh_MX_1.00u -> ScottoKeebs_Hotswap:Hotswap_MX_1.50u
- MX55, MX64: footprint PCM_Switch_Keyboard_Hotswap_Kailh:SW_Hotswap_Kailh_MX_2.25u -> ScottoKeebs_Hotswap:Hotswap_MX_1.00u
- MX56: footprint PCM_Switch_Keyboard_Hotswap_Kailh:SW_Hotswap_Kailh_MX_1.00u -> ScottoKeebs_Hotswap:Hotswap_MX_2.25u
- MX61: footprint PCM_Switch_Keyboard_Hotswap_Kailh:SW_Hotswap_Kailh_MX_1.75u -> ScottoKeebs_Hotswap:Hotswap_MX_1.00u
- MX62: footprint PCM_Switch_Keyboard_Hotswap_Kailh:SW_Hotswap_Kailh_MX_1.00u -> ScottoKeebs_Hotswap:Hotswap_MX_1.75u
- MX65: footprint PCM_Switch_Keyboard_Hotswap_Kailh:SW_Hotswap_Kailh_MX_1.25u -> ScottoKeebs_Hotswap:Hotswap_MX_2.25u
- MX68: footprint PCM_Switch_Keyboard_Hotswap_Kailh:SW_Hotswap_Kailh_MX_1.00u -> ScottoKeebs_Hotswap:Hotswap_MX_1.25u
- MX9: footprint PCM_Switch_Keyboard_Hotswap_Kailh:SW_Hotswap_Kailh_MX_1.50u -> ScottoKeebs_Hotswap:Hotswap_MX_1.50u
- OLED1: value OLED_128x32 -> locked
- S22: footprint PCM_marbastlib-mx:STAB_MX_2u -> ScottoKeebs_Stabilizer:Stabilizer_MX_2.00u
- U1: footprint PCM_marbastlib-xp-promicroish:ProMicro_USBup -> winkeebs:RP2040_ProMicro_USBup
- U2: footprint PCM_marbastlib-xp-promicroish:ProMicro_USBdn -> winkeebs:RP2040_ProMicro_USBdn
- moved H1 361.1 mm to (78.2, 61.8)
- moved H2 339.1 mm to (191.1, 48.8)
- moved H4 310.8 mm to (134.5, 107.7)
- moved H3 288.0 mm to (190.5, 107.2)
- moved MX41 166.9 mm to (439.4, 58.0), turned to -14 degrees
- moved D41 166.2 mm to (447.6, 59.7), turned to 76 degrees
- moved LED41 165.9 mm to (438.1, 62.9), turned to 166 degrees
- moved MX49 163.3 mm to (434.8, 76.5), turned to -14 degrees
- moved MX63 163.2 mm to (425.6, 113.5), turned to -14 degrees
- moved D63 162.6 mm to (433.8, 115.1), turned to 76 degrees
- moved D49 162.5 mm to (443.0, 78.1), turned to 76 degrees
- moved LED49 162.3 mm to (433.5, 81.4), turned to 166 degrees
- moved LED63 162.2 mm to (424.3, 118.4), turned to 166 degrees
- moved MX56 155.0 mm to (423.2, 93.2), turned to -14 degrees
- moved D56 154.2 mm to (431.4, 94.9), turned to 76 degrees
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- renumbered J1 to locked
Connections:
- D33 pad 1: RowR 0 -> RowL 4
- D41 pad 1: RowR 1 -> RowR 0
- D49 pad 1: RowR 2 -> RowR 1
- D56 pad 1: RowR 3 -> RowR 2
- D63 pad 1: RowR 4 -> RowR 3
- ESD1 pad 4: Net-(ESD1-IO3) -> DATA1
- ESD2 pad 4: Net-(ESD2-IO3) -> DATA2
- LED22 pad 2: Net-(LED22-DOUT) -> unconnected-(LED22-DOUT-Pad2)
- LED28 pad 1: +5V -> unconnected-(LED28-VDD-Pad1)
- LED28 pad 2: Net-(LED28-DOUT) -> unconnected-(LED28-DOUT-Pad2)
- LED28 pad 3: Net-(LED22-DOUT) -> unconnected-(LED28-DIN-Pad3)
- LED29 pad 2: Net-(LED29-DOUT) -> unconnected-(LED29-DOUT-Pad2)
- LED29 pad 3: Net-(LED28-DOUT) -> unconnected-(LED29-DIN-Pad3)
- LED30 pad 3: Net-(LED29-DOUT) -> unconnected-(LED30-DIN-Pad3)
- LED32 pad 2: unconnected-(LED32-DOUT-Pad2) -> Net-(LED32-DOUT)
- LED33 pad 2: Net-(LED33-DOUT) -> unconnected-(LED33-DOUT-Pad2)
- LED33 pad 3: LED2 -> Net-(LED32-DOUT)
- LED34 pad 3: Net-(LED33-DOUT) -> LED2
- LED41 pad 3: Net-(LED41-DIN) -> Net-(LED40-DOUT)
- LED42 pad 2: Net-(LED41-DIN) -> Net-(LED42-DOUT)
- LED48 pad 3: Net-(LED40-DOUT) -> Net-(LED48-DIN)
- LED49 pad 2: Net-(LED49-DOUT) -> Net-(LED48-DIN)
- LED50 pad 3: Net-(LED49-DOUT) -> Net-(LED42-DOUT)
- LED56 pad 3: Net-(LED56-DIN) -> Net-(LED55-DOUT)
- LED57 pad 2: Net-(LED56-DIN) -> Net-(LED57-DOUT)
- LED62 pad 3: Net-(LED55-DOUT) -> Net-(LED62-DIN)
- LED63 pad 2: Net-(LED63-DOUT) -> Net-(LED62-DIN)
- LED64 pad 3: Net-(LED63-DOUT) -> Net-(LED57-DOUT)
- LED70 pad 2: unconnected-(LED70-DOUT-Pad2) -> Net-(LED70-DOUT)
- MX28 pad 1: ColL 1 -> ColL 0
- MX29 pad 1: ColL 3 -> ColL 1
- MX30 pad 1: ColL 4 -> ColL 3
- MX31 pad 1: ColL 5 -> ColL 4
- MX32 pad 1: ColL 6 -> ColL 5
- MX33 pad 1: ColR 0 -> ColL 6
- MX34 pad 1: ColR 1 -> ColR 0
- MX35 pad 1: ColR 2 -> ColR 1
- MX36 pad 1: ColR 3 -> ColR 2
- MX37 pad 1: ColR 4 -> ColR 3
- MX38 pad 1: ColR 5 -> ColR 4
- MX39 pad 1: ColR 6 -> ColR 5
- MX40 pad 1: ColR 7 -> ColR 6
- MX41 pad 1: ColR 0 -> ColR 7
- MX42 pad 1: ColR 1 -> ColR 0
- MX43 pad 1: ColR 2 -> ColR 1
- MX44 pad 1: ColR 3 -> ColR 2
- MX45 pad 1: ColR 4 -> ColR 3
- MX46 pad 1: ColR 5 -> ColR 4
- MX47 pad 1: ColR 6 -> ColR 5
- MX48 pad 1: ColR 7 -> ColR 6
- MX49 pad 1: ColR 0 -> ColR 7
- MX50 pad 1: ColR 1 -> ColR 0
- MX51 pad 1: ColR 2 -> ColR 1
- MX52 pad 1: ColR 3 -> ColR 2
- MX53 pad 1: ColR 4 -> ColR 3
- MX54 pad 1: ColR 5 -> ColR 4
- MX55 pad 1: ColR 6 -> ColR 5
- MX56 pad 1: ColR 0 -> ColR 6
- MX57 pad 1: ColR 1 -> ColR 0
- MX58 pad 1: ColR 2 -> ColR 1
- MX59 pad 1: ColR 3 -> ColR 2
- MX60 pad 1: ColR 4 -> ColR 3
- MX61 pad 1: ColR 5 -> ColR 4
- MX62 pad 1: ColR 6 -> ColR 5
- MX63 pad 1: ColR 0 -> ColR 6
- MX64 pad 1: ColR 1 -> ColR 0
- MX65 pad 1: ColR 2 -> ColR 1
- MX66 pad 1: ColR 3 -> ColR 2
- MX67 pad 1: ColR 4 -> ColR 3
- MX68 pad 1: ColR 5 -> ColR 4
- MX69 pad 1: ColR 6 -> ColR 5
- MX70 pad 1: ColR 7 -> ColR 6
- U1 pad 1: Net-(ESD1-IO3) -> LED1
- U1 pad 10: RowL 3 -> unconnected-(U1-Pad10)
- U1 pad 11: RowL 4 -> unconnected-(U1-Pad11)
- U1 pad 12: VCC -> ROTS
- U1 pad 13: +5V -> ROTB
- U1 pad 14: GND -> ROTA
- U1 pad 15: Reset1 -> unconnected-(U1-Pad15)
- U1 pad 16: VCC -> unconnected-(U1-Pad16)
- U1 pad 18: ColL 0 -> unconnected-(U1-Pad18)
- U1 pad 2: LED1 -> SDA1
- U1 pad 20: ColL 2 -> ColL 4
- U1 pad 21: ColL 3 -> ColL 6
- U1 pad 22: ColL 4 -> ColL 3
- U1 pad 24: ColL 6 -> unconnected-(U1-Pad24)
- U1 pad 3: GND -> SCL1
- U1 pad 4: GND -> RowL 0
- U1 pad 5: SDA1 -> RowL 1
- U1 pad 6: SCL1 -> RowL 2
- U1 pad 7: RowL 0 -> RowL 3
- U1 pad 8: RowL 1 -> RowL 4
- U1 pad 9: RowL 2 -> VCC
- U2 pad 1: Net-(ESD2-IO3) -> LED2
- U2 pad 10: RowR 3 -> unconnected-(U2-Pad10)
- U2 pad 11: RowR 4 -> unconnected-(U2-Pad11)
- U2 pad 12: GND -> unconnected-(U2-Pad12)
- U2 pad 13: RAW2 -> unconnected-(U2-Pad13)
- U2 pad 14: GND -> unconnected-(U2-Pad14)
- U2 pad 15: Reset2 -> unconnected-(U2-Pad15)
- U2 pad 16: VCC -> unconnected-(U2-Pad16)
- U2 pad 18: ColR 1 -> unconnected-(U2-Pad18)
- U2 pad 2: LED2 -> SDA2
- U2 pad 20: ColR 3 -> ColR 5
- U2 pad 21: ColR 4 -> ColR 7
- U2 pad 22: ColR 5 -> ColR 4
- U2 pad 24: ColR 7 -> unconnected-(U2-Pad24)
- U2 pad 3: GND -> SCL2
- U2 pad 4: GND -> RowR 0
- U2 pad 5: SDA2 -> RowR 1
- U2 pad 6: SCL2 -> RowR 2
- U2 pad 7: RowR 0 -> RowR 3
- U2 pad 8: RowR 1 -> RowR 4
- U2 pad 9: RowR 2 -> GND
Routing:
- net GND: track 0.00 -> 179.9 mm, vias 0 -> 9
- net VCC: track 0.00 -> 114.4 mm, vias 0 -> 5
- net RowL 4: track 171.0 -> 235.8 mm, vias 8 -> 10
- net RowR 3: track 156.7 -> 202.7 mm
- net ColL 6: track 118.9 -> 83.6 mm, vias 3 -> 2
- net RowR 4: track 191.4 -> 226.3 mm, vias 14 -> 12
- net DATA1: track 0.00 -> 32.5 mm, vias 0 -> 2
- net ColL 2: track 95.2 -> 63.1 mm, vias 1 -> 0
- net RowL 0: track 144.6 -> 175.6 mm, vias 9 -> 12
- net +5V: track 0.00 -> 31.0 mm, vias 0 -> 2
- net SDA2: track 0.00 -> 28.9 mm, vias 0 -> 1
- net RowR 2: track 154.3 -> 183.1 mm
- net DATA2: track 0.00 -> 28.1 mm, vias 0 -> 1
- net SDA1: track 0.00 -> 26.2 mm
- net SCL2: track 0.00 -> 25.5 mm, vias 0 -> 1
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Other:
- board size 4.1 x 3.8 mm -> 422.1 x 120.4 mm
