File: pcb/_autosave-Win-split.kicad_sch (KiCad schematic)
At the start: 242 parts, among them J1 Conn_01x04_Socket, J2 Conn_01x04_Socket, SW1 ROT_SKYLOONG_HS, SW2 ROT_SKYLOONG_HS, U1 RP2040_ProMicro, U2 RP2040_ProMicro

Commit message: pre-del button
Parts:
- removed SW2: ROT_SKYLOONG_HS, PCM_marbastlib-various:ROT_SKYLOONG_HS-Switch, symbol PCM_marbastlib-various:ROT_SKYLOONG_HS-Switch
Connections:
- net GND: no longer SW1.C
Other:
- moved on the sheet: D28, MX28
Changed lines of the file:
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@@
   (junction (at 742.95 55.88) (diameter 0) (color 0 0 0 0)
   )
+  (junction (at 207.01 166.37) (diameter 0) (color 0 0 0 0)
+  )
   (junction (at 717.55 132.08) (diameter 0) (color 0 0 0 0)
   )
@@
   (junction (at 671.83 93.98) (diameter 0) (color 0 0 0 0)
   )
-  (junction (at 48.26 106.68) (diameter 0) (color 0 0 0 0)
-  )
   (junction (at 278.13 52.07) (diameter 0) (color 0 0 0 0)
   )
@@
   (junction (at 659.13 330.2) (diameter 0) (color 0 0 0 0)
   )
-  (junction (at 205.74 166.37) (diameter 0) (color 0 0 0 0)
-  )
   (junction (at 692.15 81.28) (diameter 0) (color 0 0 0 0)
   )
@@
     (stroke (width 0) (type default))
   )
-  (wire (pts (xy 48.26 100.33) (xy 48.26 106.68))
-    (stroke (width 0) (type default))
-  )
   (wire (pts (xy 565.15 55.88) (xy 565.15 81.28))
     (stroke (width 0) (type default))
@@
     (stroke (width 0) (type default))
   )
-  (wire (pts (xy 58.42 100.33) (xy 48.26 100.33))
-    (stroke (width 0) (type default))
-  )
   (wire (pts (xy 659.13 284.48) (xy 659.13 289.56))
     (stroke (width 0) (type default))
@@
     (stroke (width 0) (type default))
   )
-  (wire (pts (xy 201.93 102.87) (xy 200.66 102.87))
-    (stroke (width 0) (type default))
-  )
   (wire (pts (xy 621.03 68.58) (xy 646.43 68.58))
     (stroke (width 0) (type default))
@@
     (stroke (width 0) (type default))
   )
-  (wire (pts (xy 26.67 100.33) (xy 16.51 100.33))
-    (stroke (width 0) (type default))
-  )
   (wire (pts (xy 60.96 46.99) (xy 62.23 46.99))
     (stroke (width 0) (type default))
@@
     (stroke (width 0) (type default))
   )
-  (wire (pts (xy 200.66 102.87) (xy 200.66 153.67))
+  (wire (pts (xy 201.93 102.87) (xy 201.93 153.67))
     (stroke (width 0) (type default))
   )
@@
     (stroke (width 0) (type default))
   )
-  (wire (pts (xy 189.23 166.37) (xy 205.74 166.37))
-    (stroke (width 0) (type default))
-  )
   (wire (pts (xy 646.43 93.98) (xy 671.83 93.98))
     (stroke (width 0) (type default))
@@
     (stroke (width 0) (type default))
   )
-  (wire (pts (xy 16.51 106.68) (xy 48.26 106.68))
-    (stroke (width 0) (type default))
-  )
   (wire (pts (xy 62.23 44.45) (xy 60.96 44.45))
     (stroke (width 0) (type default))
@@
     (stroke (width 0) (type default))
   )
-  (wire (pts (xy 205.74 166.37) (xy 232.41 166.37))
+  (wire (pts (xy 189.23 166.37) (xy 207.01 166.37))
     (stroke (width 0) (type default))
   )
@@
     (stroke (width 0) (type dash_dot))
   )
-  (wire (pts (xy 16.51 100.33) (xy 16.51 106.68))
-    (stroke (width 0) (type default))
-  )
   (wire (pts (xy 334.01 140.97) (xy 359.41 140.97))
     (stroke (width 0) (type default))
@@
     (stroke (width 0) (type default))
   )
+  (wire (pts (xy 207.01 166.37) (xy 232.41 166.37))
+    (stroke (width 0) (type default))
+  )
   (wire (pts (xy 173.99 219.71) (xy 191.77 219.71))
     (stroke (width 0) (type default))
@@
     )
   )
-  (global_label "ROTS" (shape input) (at 73.66 97.79 0) (fields_autoplaced)
-    (effects (font (size 1.27 1.27)) (justify left))
-    (property "Intersheetrefs" "${INTERSHEET_REFS}" (at 81.4228 97.79 0)
-      (effects (font (size 1.27 1.27)) (justify left) hide)
-    )
-  )
   (global_label "RowR 1" (shape input) (at 440.69 54.61 0) (fields_autoplaced)
     (effects (font (size 1.27 1.27)) (justify left))
@@
     )
   )
-  (global_label "ROTA" (shape input) (at 58.42 97.79 180) (fields_autoplaced)
-    (effects (font (size 1.27 1.27)) (justify right))
-    (property "Intersheetrefs" "${INTERSHEET_REFS}" (at 50.7781 97.79 0)
-      (effects (font (size 1.27 1.27)) (justify right) hide)
-    )
-  )
   (global_label "ColL 1" (shape input) (at 227.33 39.37 90) (fields_autoplaced)
     (effects (font (size 1.27 1.27)) (justify left))
@@
     )
   )
-  (global_label "ROTB" (shape input) (at 58.42 102.87 180) (fields_autoplaced)
-    (effects (font (size 1.27 1.27)) (justify right))
-    (property "Intersheetrefs" "${INTERSHEET_REFS}" (at 50.5967 102.87 0)
-      (effects (font (size 1.27 1.27)) (justify right) hide)
-    )
-  )
   (global_label "ColL 1" (shape input) (at 35.56 54.61 180) (fields_autoplaced)
     (effects (font (size 1.27 1.27)) (justify right))
@@
     )
   )
-  (symbol (lib_id "ScottoKeebs:Placeholder_Diode") (at 205.74 162.56 90) (unit 1)
+  (symbol (lib_id "ScottoKeebs:Placeholder_Diode") (at 207.01 162.56 90) (unit 1)
     (in_bom yes) (on_board yes) (dnp no) (fields_autoplaced)
-    (property "Reference" "D28" (at 208.28 161.29 90)
+    (property "Reference" "D28" (at 209.55 161.29 90)
       (effects (font (size 1.27 1.27)) (justify right))
     )
-    (property "Value" "Diode" (at 208.28 163.83 90)
+    (property "Value" "Diode" (at 209.55 163.83 90)
       (effects (font (size 1.27 1.27)) (justify right) hide)
     )
-    (property "Footprint" "ScottoKeebs_Components:Diode_SOD-123" (at 205.74 162.56 0)
+    (property "Footprint" "ScottoKeebs_Components:Diode_SOD-123" (at 207.01 162.56 0)
       (effects (font (size 1.27 1.27)) hide)
     )
-    (property "Datasheet" "" (at 205.74 162.56 0)
+    (property "Datasheet" "" (at 207.01 162.56 0)
       (effects (font (size 1.27 1.27)) hide)
     )
-    (property "Sim.Device" "D" (at 205.74 162.56 0)
+    (property "Sim.Device" "D" (at 207.01 162.56 0)
       (effects (font (size 1.27 1.27)) hide)
     )
-    (property "Sim.Pins" "1=K 2=A" (at 205.74 162.56 0)
+    (property "Sim.Pins" "1=K 2=A" (at 207.01 162.56 0)
       (effects (font (size 1.27 1.27)) hide)
     )
-    (property "LCSC" "C2972760" (at 205.74 162.56 0)
+    (property "LCSC" "C2972760" (at 207.01 162.56 0)
       (effects (font (size 1.27 1.27)) hide)
     )
@@
     )
   )
-  (symbol (lib_name "GND_2") (lib_id "power:GND") (at 48.26 106.68 0) (mirror y) (unit 1)
-    (in_bom yes) (on_board yes) (dnp no) (fields_autoplaced)
-    (property "Reference" "#PWR031" (at 48.26 113.03 0)
-      (effects (font (size 1.27 1.27)) hide)
-    )
-    (property "Value" "GND" (at 48.26 110.49 90)
-      (effects (font (size 1.27 1.27)) (justify right) hide)
-    )
-    (property "Footprint" "" (at 48.26 106.68 0)
-      (effects (font (size 1.27 1.27)) hide)
-    )
-    (property "Datasheet" "" (at 48.26 106.68 0)
-      (effects (font (size 1.27 1.27)) hide)
-    )
-    (pin "1")
-    (instances
-      (project "Win-split"
-        (path "/49098896-502f-4162-bad5-517f7d921ed4"
-          (reference "#PWR031") (unit 1)
-        )
-      )
-    )
-  )
   (symbol (lib_id "ScottoKeebs:Placeholder_Diode") (at 671.83 166.37 90) (unit 1)
     (in_bom yes) (on_board yes) (dnp no) (fields_autoplaced)
@@
     )
   )
-  (symbol (lib_id "PCM_marbastlib-various:ROT_SKYLOONG_HS-Switch") (at 66.04 100.33 0) (unit 1)
-    (in_bom no) (on_board yes) (dnp no)
-    (property "Reference" "SW2" (at 66.04 90.17 0)
-      (effects (font (size 1.27 1.27)))
-    )
-    (property "Value" "ROT_SKYLOONG_HS" (at 66.04 92.71 0)
-      (effects (font (size 1.27 1.27)))
-    )
-    (property "Footprint" "PCM_marbastlib-various:ROT_SKYLOONG_HS-Switch" (at 66.04 100.33 0)
-      (effects (font (size 1.27 1.27)) hide)
-    )
-    (property "Datasheet" "https://skyloong.vip/products/abs-hot-swappable-knobs-madule" (at 66.04 100.33 0)
-      (effects (font (size 1.27 1.27)) hide)
-    )
-    (pin "B")
-    (pin "C")
-    (pin "A")
-    (pin "S")
-    (instances
-      (project "Win-split"
-        (path "/49098896-502f-4162-bad5-517f7d921ed4"
-          (reference "SW2") (unit 1)
-        )
-      )
-    )
-  )
   (symbol (lib_id "PCM_marbastlib-mx:MX_SK6812MINI-E") (at 608.33 297.18 180) (unit 1)
     (in_bom yes) (on_board yes) (dnp no)
@@
     )
   )
-  (symbol (lib_id "PCM_marbastlib-mx:MX_SW_HS") (at 203.2 156.21 0) (unit 1)
+  (symbol (lib_id "PCM_marbastlib-mx:MX_SW_HS") (at 204.47 156.21 0) (unit 1)
     (in_bom yes) (on_board yes) (dnp no)
-    (property "Reference" "MX28" (at 203.2 151.13 0)
+    (property "Reference" "MX28" (at 204.47 151.13 0)
       (effects (font (size 1.27 1.27)))
     )
-    (property "Value" "MX_SW_HS" (at 203.2 151.13 0)
+    (property "Value" "MX_SW_HS" (at 204.47 151.13 0)
       (effects (font (size 1.27 1.27)) hide)
     )
-    (property "Footprint" "ScottoKeebs_Hotswap:Hotswap_MX_1.00u" (at 203.2 156.21 0)
+    (property "Footprint" "ScottoKeebs_Hotswap:Hotswap_MX_1.00u" (at 204.47 156.21 0)
       (effects (font (size 1.27 1.27)) hide)
     )
-    (property "Datasheet" "~" (at 203.2 156.21 0)
+    (property "Datasheet" "~" (at 204.47 156.21 0)
       (effects (font (size 1.27 1.27)) hide)
     )
