File: pcb/left/Win-split-left.kicad_pcb (KiCad board)
At the start: 2 copper layers, 422.1 x 120.4 mm, 121 parts, among them J1 Conn_01x04_Socket, Q1 Q_PMOS_GSD, SW8 ROT_SKYLOONG_HS, U1 RP2040_ProMicro, U3 74AHCT1G125

Commit message: kicad 7
Parts:
- added C1: 100nF, Capacitor_SMD:C_0402_1005Metric, B.Cu at (117.4, 97.8)
- added C10: 100nF, Capacitor_SMD:C_0402_1005Metric, B.Cu at (154.3, 108.2)
- added C100: 100nF, Capacitor_SMD:C_0402_1005Metric, B.Cu at (246.3, 79.7)
- added C11: 100nF, Capacitor_SMD:C_0402_1005Metric, B.Cu at (174.2, 104.0)
- added C12: 100nF, Capacitor_SMD:C_0402_1005Metric, B.Cu at (193.2, 101.7)
- added C13: 100nF, Capacitor_SMD:C_0402_1005Metric, B.Cu at (212.3, 104.0)
- added C14: 100nF, Capacitor_SMD:C_0402_1005Metric, B.Cu at (231.3, 106.4)
- added C15: 100nF, Capacitor_SMD:C_0402_1005Metric, B.Cu at (89.6, 124.4)
- added C16: 100nF, Capacitor_SMD:C_0402_1005Metric, B.Cu at (128.9, 134.2)
- added C17: 100nF, Capacitor_SMD:C_0402_1005Metric, B.Cu at (154.3, 127.9)
- added C18: 100nF, Capacitor_SMD:C_0402_1005Metric, B.Cu at (174.2, 123.0)
- added C19: 100nF, Capacitor_SMD:C_0402_1005Metric, B.Cu at (193.2, 120.7)
- added C20: 100nF, Capacitor_SMD:C_0402_1005Metric, B.Cu at (212.3, 123.0)
- added C21: 100nF, Capacitor_SMD:C_0402_1005Metric, B.Cu at (231.3, 125.5)
- added C22: 100nF, Capacitor_SMD:C_0402_1005Metric, B.Cu at (94.3, 142.9)
- added C23: 100nF, Capacitor_SMD:C_0402_1005Metric, B.Cu at (126.6, 154.4)
- added C24: 100nF, Capacitor_SMD:C_0402_1005Metric, B.Cu at (154.3, 147.5)
- added C25: 100nF, Capacitor_SMD:C_0402_1005Metric, B.Cu at (174.2, 142.1)
- added C26: 100nF, Capacitor_SMD:C_0402_1005Metric, B.Cu at (193.2, 139.8)
- added C27: 100nF, Capacitor_SMD:C_0402_1005Metric, B.Cu at (212.3, 142.1)
- added C28: 100nF, Capacitor_SMD:C_0402_1005Metric, B.Cu at (231.3, 144.5)
- added C29: 100nF, Capacitor_SMD:C_0402_1005Metric, B.Cu at (89.6, 183.3)
- added C3: 100nF, Capacitor_SMD:C_0402_1005Metric, B.Cu at (154.4, 88.6)
- added C30: 100nF, Capacitor_SMD:C_0402_1005Metric, B.Cu at (133.5, 172.3)
- added C31: 100nF, Capacitor_SMD:C_0402_1005Metric, B.Cu at (186.1, 161.1)
- added C32: 100nF, Capacitor_SMD:C_0402_1005Metric, B.Cu at (209.9, 161.1)
- added C33: 100nF, Capacitor_SMD:C_0402_1005Metric, B.Cu at (240.9, 163.6)
- added C34: 100nF, Capacitor_SMD:C_0402_1005Metric, B.Cu at (250.4, 144.5)
- added C4: 100nF, Capacitor_SMD:C_0402_1005Metric, B.Cu at (174.2, 84.9)
- added C5: 100nF, Capacitor_SMD:C_0402_1005Metric, B.Cu at (193.2, 82.6)
- added C6: 100nF, Capacitor_SMD:C_0402_1005Metric, B.Cu at (212.3, 84.9)
- added C7: 100nF, Capacitor_SMD:C_0402_1005Metric, B.Cu at (231.3, 87.4)
- added C8: 100nF, Capacitor_SMD:C_0402_1005Metric, B.Cu at (71.2, 109.3)
- added C9: 100nF, Capacitor_SMD:C_0402_1005Metric, B.Cu at (131.2, 114.0)
- D1, D10, D11, D12, D13, D14, D15, D16, D17, D18, D19, D2, D20, D21, D22, D23, D24, D25, D26, D27, D28, D29, D3, D30, D31, D32, D33, D34, D4, D5, D6, D7, D8, D9: footprint ScottoKeebs_Components:Diode_SOD-123 -> winkeebs:Diode_SOD-123
- LED1, LED15, LED16, LED17, LED18, LED19, LED2, LED20, LED21, LED29, LED3, LED30, LED31, LED32, LED33, LED34, LED4, LED5, LED6, LED7: footprint winkeebs:LED_MX_6028R-ROT -> PCM_marbastlib-mx:LED_MX_6028R
- LED10, LED11, LED12, LED13, LED14, LED22, LED23, LED24, LED25, LED26, LED27, LED28, LED8, LED9: footprint winkeebs:LED_MX_6028R -> PCM_marbastlib-mx:LED_MX_6028R-ROT
- MX1, MX10, MX11, MX12, MX13, MX14, MX15, MX17, MX18, MX19, MX2, MX20, MX21, MX22, MX24, MX25, MX26, MX27, MX28, MX29, MX3, MX34, MX4, MX5, MX6, MX7, MX8: footprint ScottoKeebs_Hotswap:Hotswap_MX_Plated_1.00u -> winkeebs:SW_MX_HS_CPG151101S11_1u; moved to B.Cu
- MX16: footprint ScottoKeebs_Hotswap:Hotswap_MX_Plated_1.75u -> winkeebs:SW_MX_HS_CPG151101S11_1.75u; moved to B.Cu
- MX23, MX33: footprint ScottoKeebs_Hotswap:Hotswap_MX_Plated_2.00u -> winkeebs:SW_MX_HS_CPG151101S11_1u; moved to B.Cu
- MX30, MX31, MX32: footprint ScottoKeebs_Hotswap:Hotswap_MX_1.25u -> winkeebs:SW_MX_HS_CPG151101S11_1.25u; moved to B.Cu
- MX9: footprint ScottoKeebs_Hotswap:Hotswap_MX_Plated_1.50u -> winkeebs:SW_MX_HS_CPG151101S11_1.5u; moved to B.Cu
- moved H1 109.4 mm to (243.6, 92.6)
- moved C2 91.4 mm to (135.9, 93.2), turned to -166 degrees
- moved Reset1 35.4 mm to (271.8, 100.0)
- moved ESD1 35.4 mm to (271.9, 93.1), turned to -135 degrees
- moved TRRS1 35.4 mm to (271.8, 75.5)
- moved D6 35.0 mm to (226.0, 80.6)
- moved MX6 35.0 mm to (217.4, 80.6), turned to 180 degrees
- moved D9 35.0 mm to (143.5, 106.5)
- moved MX26 35.0 mm to (198.3, 135.4), turned to 180 degrees
- moved D11 35.0 mm to (187.9, 99.6)
- moved LED6 35.0 mm to (217.4, 85.7)
- moved MX24 35.0 mm to (158.2, 142.1), turned to -166 degrees
- moved MX20 35.0 mm to (217.4, 118.7), turned to 180 degrees
- moved MX30 35.0 mm to (137.4, 166.9), turned to -166 degrees
- moved MX8 35.0 mm to (75.1, 103.9), turned to -166 degrees
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Connections:
- C2 pad 1: GND -> +5V
- C2 pad 2: +5V -> GND
Routing:
- net Net-(Q1-G): track 18.5 -> 0.00 mm
- net Net-(D16-A): track 9.58 -> 4.47 mm
- net Net-(D21-A): track 9.58 -> 4.47 mm
- net Net-(D23-A): track 9.58 -> 4.47 mm
- net Net-(D10-A): track 9.58 -> 4.47 mm
- net Net-(D24-A): track 9.58 -> 4.47 mm
- net Net-(D9-A): track 9.58 -> 4.47 mm
- net Net-(D33-A): track 9.58 -> 4.47 mm
- net Net-(D18-A): track 9.58 -> 4.47 mm
- net Net-(D29-A): track 9.58 -> 4.47 mm
- net SW/MX: track 9.58 -> 4.47 mm
- net Net-(D5-A): track 9.58 -> 4.47 mm
- net Net-(D3-A): track 9.58 -> 4.47 mm
- net Net-(D22-A): track 9.58 -> 4.47 mm
- net Net-(D12-A): track 9.58 -> 4.47 mm
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Other:
- board size 422.1 x 120.4 mm -> 4.1 x 3.8 mm

Commit message: before rounding tracks in left side
Parts:
- added H6: MountingHole_Pad, winkeebs:HOLE_M2, F.Cu at (189.6, 164.3)
- added H7: MountingHole_Pad, winkeebs:HOLE_M2, F.Cu at (246.0, 145.6)
- added H8: MountingHole_Pad, winkeebs:HOLE_M2, F.Cu at (288.8, 156.4)
- ESD1, Q1, R1, R2: moved to B.Cu
- LED15, LED34: footprint PCM_marbastlib-mx:LED_MX_6028R -> PCM_marbastlib-mx:LED_MX_6028R-ROT
- LED22, LED8: footprint PCM_marbastlib-mx:LED_MX_6028R-ROT -> PCM_marbastlib-mx:LED_MX_6028R
- moved H4 243.4 mm to (122.0, 181.9)
- moved H3 223.4 mm to (108.9, 124.9)
- moved H5 175.7 mm to (165.7, 131.7)
- moved H2 150.6 mm to (186.5, 107.9)
- moved U3 37.3 mm to (276.1, 99.3)
- moved C100 37.3 mm to (276.1, 102.1)
- moved C27 34.3 mm to (241.6, 159.8), turned to 0 degrees
- moved C14 34.3 mm to (260.6, 124.2), turned to 0 degrees
- moved C13 34.2 mm to (241.6, 121.6), turned to 0 degrees
- moved C28 34.2 mm to (260.6, 162.2), turned to 0 degrees
- moved C34 34.2 mm to (279.6, 162.3), turned to 0 degrees
- moved C25 34.2 mm to (203.4, 159.8), turned to 0 degrees
- moved C12 34.1 mm to (222.4, 119.4), turned to 0 degrees
- moved C11 34.1 mm to (203.4, 121.6), turned to 0 degrees
- moved C26 34.1 mm to (222.4, 157.4), turned to 0 degrees
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Connections:
- C15 pad 1: +5V -> GND
- C15 pad 2: GND -> +5V
- LED16 pad 2: Net-(LED15-DIN) -> Net-(LED16-DOUT)
- LED22 pad 3: Net-(LED15-DOUT) -> Net-(LED16-DOUT)
- LED8 pad 2: Net-(LED8-DOUT) -> Net-(LED15-DIN)
- LED9 pad 3: Net-(LED8-DOUT) -> Net-(LED15-DOUT)
- TRRS1 pad 1: VCC -> GND
- TRRS1 pad 2: unconnected-(TRRS1-TIP-Pad2) -> VCC
- TRRS1 pad 3: Net-(ESD1-IO1) -> unconnected-(TRRS1-RING1-Pad3)
- TRRS1 pad 4: GND -> Net-(ESD1-IO1)
- U1 pad 20: COL4 -> COL2
- U1 pad 21: COL6 -> COL0
- U1 pad 23: COL5 -> COL1
- U1 pad 26: COL2 -> COL4
- U1 pad 27: COL1 -> COL5
- U1 pad 28: COL0 -> COL6
Routing:
- net +5V: track 0.00 -> 964.6 mm, vias 0 -> 8
- net COL0: track 0.00 -> 361.9 mm, vias 0 -> 1
- net COL1: track 0.00 -> 251.9 mm, vias 0 -> 2
- net ROW4: track 0.00 -> 231.8 mm, vias 0 -> 1
- net VCC: track 0.00 -> 228.4 mm, vias 0 -> 2
- net COL3: track 0.00 -> 208.7 mm, vias 0 -> 2
- net COL2: track 0.00 -> 205.0 mm, vias 0 -> 2
- net COL4: track 0.00 -> 198.6 mm, vias 0 -> 2
- net COL5: track 0.00 -> 195.8 mm, vias 0 -> 2
- net ROW3: track 0.00 -> 194.9 mm, vias 0 -> 3
- net ROTA: track 0.00 -> 192.0 mm, vias 0 -> 5
- net ROTB: track 0.00 -> 190.2 mm, vias 0 -> 4
- net ROW2: track 0.00 -> 187.0 mm, vias 0 -> 3
- net ROW1: track 0.00 -> 186.9 mm, vias 0 -> 2
- net ROW0: track 0.00 -> 145.3 mm, vias 0 -> 1
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- added copper zone on B.Cu, net GND
- added copper zone on F.Cu, net GND
Other:
- board size 4.1 x 3.8 mm -> 213.2 x 120.4 mm
