File: pcb/left/Win-split-left.kicad_pcb (KiCad board)
At the start: 2 copper layers, 4.1 x 3.8 mm, 155 parts, among them J1 Conn_01x04_Socket, Q1 Q_PMOS_GSD, SW8 ROT_SKYLOONG_HS, U1 RP2040_ProMicro, U3 74AHCT1G125

Commit message: prerouting right side
Parts:
- removed OLED1: OLED_128x32, ScottoKeebs_Components:OLED_128x32
- added H6: MountingHole_Pad, winkeebs:HOLE_M2, F.Cu at (197.0, 167.3)
- added H7: MountingHole_Pad, winkeebs:HOLE_M2, F.Cu at (253.4, 148.6)
- added H8: MountingHole_Pad, winkeebs:HOLE_M2, F.Cu at (296.2, 159.4)
- ESD1, Q1, R1, R2: moved to B.Cu
- LED15, LED34: footprint PCM_marbastlib-mx:LED_MX_6028R -> PCM_marbastlib-mx:LED_MX_6028R-ROT
- LED22, LED8: footprint PCM_marbastlib-mx:LED_MX_6028R-ROT -> PCM_marbastlib-mx:LED_MX_6028R
- moved H4 239.9 mm to (129.4, 184.8)
- moved H3 218.4 mm to (116.3, 127.9)
- moved H5 171.8 mm to (173.2, 134.6)
- moved H2 146.8 mm to (193.9, 110.9)
- moved U3 45.1 mm to (283.5, 102.3)
- moved C100 45.1 mm to (283.5, 105.1)
- moved C27 42.2 mm to (249.0, 162.8), turned to 0 degrees
- moved C14 42.1 mm to (268.0, 127.2), turned to 0 degrees
- moved C13 42.1 mm to (249.0, 124.6), turned to 0 degrees
- moved C28 42.1 mm to (268.0, 165.2), turned to 0 degrees
- moved C34 42.1 mm to (287.0, 165.2), turned to 0 degrees
- moved C25 42.1 mm to (210.8, 162.8), turned to 0 degrees
- moved C11 42.0 mm to (210.8, 124.6), turned to 0 degrees
- moved C12 42.0 mm to (229.8, 122.4), turned to 0 degrees
- moved C26 42.0 mm to (229.8, 160.4), turned to 0 degrees
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Connections:
- C15 pad 1: +5V -> GND
- C15 pad 2: GND -> +5V
- LED16 pad 2: Net-(LED15-DIN) -> Net-(LED16-DOUT)
- LED22 pad 3: Net-(LED15-DOUT) -> Net-(LED16-DOUT)
- LED8 pad 2: Net-(LED8-DOUT) -> Net-(LED15-DIN)
- LED9 pad 3: Net-(LED8-DOUT) -> Net-(LED15-DOUT)
- TRRS1 pad 1: VCC -> GND
- TRRS1 pad 2: unconnected-(TRRS1-TIP-Pad2) -> VCC
- TRRS1 pad 3: Net-(ESD1-IO1) -> unconnected-(TRRS1-RING1-Pad3)
- TRRS1 pad 4: GND -> Net-(ESD1-IO1)
- U1 pad 20: COL4 -> COL2
- U1 pad 21: COL6 -> COL0
- U1 pad 23: COL5 -> COL1
- U1 pad 26: COL2 -> COL4
- U1 pad 27: COL1 -> COL5
- U1 pad 28: COL0 -> COL6
Routing:
- net +5V: track 0.00 -> 972.4 mm, vias 0 -> 8
- net COL0: track 0.00 -> 362.6 mm, vias 0 -> 1
- net COL1: track 0.00 -> 252.4 mm, vias 0 -> 2
- net ROW4: track 0.00 -> 232.6 mm, vias 0 -> 1
- net VCC: track 0.00 -> 228.8 mm, vias 0 -> 2
- net COL3: track 0.00 -> 208.8 mm, vias 0 -> 2
- net COL2: track 0.00 -> 205.2 mm, vias 0 -> 2
- net COL4: track 0.00 -> 198.7 mm, vias 0 -> 2
- net ROW3: track 0.00 -> 197.6 mm, vias 0 -> 3
- net COL5: track 0.00 -> 192.8 mm, vias 0 -> 2
- net ROTA: track 0.00 -> 192.0 mm, vias 0 -> 5
- net ROW1: track 0.00 -> 192.0 mm, vias 0 -> 2
- net ROTB: track 0.00 -> 190.8 mm, vias 0 -> 4
- net ROW2: track 0.00 -> 187.4 mm, vias 0 -> 3
- net ROW0: track 0.00 -> 146.9 mm, vias 0 -> 1
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- added copper zone on B.Cu, net GND
- added copper zone on F.Cu, net GND
Other:
- board size 4.1 x 3.8 mm -> 213.2 x 120.4 mm
