File: pcb/left/Win-split-left.kicad_sch (KiCad schematic)
At the start: 155 parts, among them J1 Conn_01x04_Socket, Q1 Q_PMOS_GSD, SW8 ROT_SKYLOONG_HS, U1 RP2040_ProMicro, U3 74AHCT1G125

Commit message: kicad 7
Parts:
- D1, D10, D11, D12, D13, D14, D15, D16, D17, D18, D19, D2, D20, D21, D22, D23, D24, D25, D26, D27, D28, D29, D3, D30, D31, D32, D33, D34, D4, D5, D6, D7, D8, D9: footprint ScottoKeebs_Components:Diode_SOD-123 -> winkeebs:Diode_SOD-123
- LED1, LED15, LED16, LED17, LED18, LED19, LED2, LED20, LED21, LED29, LED3, LED30, LED31, LED32, LED33, LED34, LED4, LED5, LED6, LED7: footprint winkeebs:LED_MX_6028R-ROT -> PCM_marbastlib-mx:LED_MX_6028R
- LED10, LED11, LED12, LED13, LED14, LED22, LED23, LED24, LED25, LED26, LED27, LED28, LED8, LED9: footprint winkeebs:LED_MX_6028R -> PCM_marbastlib-mx:LED_MX_6028R-ROT
- MX1, MX10, MX11, MX12, MX13, MX14, MX15, MX17, MX18, MX19, MX2, MX20, MX21, MX22, MX23, MX24, MX25, MX26, MX27, MX28, MX29, MX3, MX33, MX34, MX4, MX5, MX6, MX7, MX8: footprint PCM_marbastlib-mx:SW_MX_HS_CPG151101S11_1u -> winkeebs:SW_MX_HS_CPG151101S11_1u
- MX16: footprint PCM_marbastlib-mx:SW_MX_HS_CPG151101S11_1u -> winkeebs:SW_MX_HS_CPG151101S11_1.75u
- MX30, MX31, MX32: footprint PCM_marbastlib-mx:SW_MX_HS_CPG151101S11_1u -> winkeebs:SW_MX_HS_CPG151101S11_1.25u
- MX9: footprint PCM_marbastlib-mx:SW_MX_HS_CPG151101S11_1u -> winkeebs:SW_MX_HS_CPG151101S11_1.5u

Commit message: before rounding tracks in left side
Parts:
- added H6, H7, H8: MountingHole_Pad, winkeebs:HOLE_M2, symbol Mechanical:MountingHole
- LED15, LED34: footprint PCM_marbastlib-mx:LED_MX_6028R -> PCM_marbastlib-mx:LED_MX_6028R-ROT
- LED22, LED8: footprint PCM_marbastlib-mx:LED_MX_6028R-ROT -> PCM_marbastlib-mx:LED_MX_6028R
Connections:
- net +5V: now also C15.2; no longer C15.1
- net COL0: now also U1.21; no longer U1.28
- net COL1: now also U1.23; no longer U1.27
- net COL2: now also U1.20; no longer U1.26
- net COL4: now also U1.26; no longer U1.20
- net COL5: now also U1.27; no longer U1.23
- net COL6: now also U1.28; no longer U1.21
- net GND: now also C15.1, TRRS1.1 (SLEEVE); no longer C15.2, TRRS1.4 (RING2)
- net VCC: now also TRRS1.2 (TIP); no longer TRRS1.1 (SLEEVE)
- net at TRRS1.3 (RING1): no longer ESD1.1 (IO1)
- net at LED9.3 (DIN): now also LED15.2 (DOUT); no longer LED8.2 (DOUT)
- net at LED22.3 (DIN): now also LED16.2 (DOUT); no longer LED15.2 (DOUT)
- net at LED15.3 (DIN): now also LED8.2 (DOUT); no longer LED16.2 (DOUT)
- new net: ESD1.1 (IO1), TRRS1.4 (RING2)
Other:
- moved on the sheet: C10, C11, C12, C13, C14, C15, C9, ESD1, H1, H2, H3, H4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
