File: pcb/right/Win-split-right.kicad_sch (KiCad schematic)
At the start: 172 parts, among them J2 Conn_01x04_Socket, U1 RP2040_ProMicro, U2 74AHCT1G125

Commit message: before rounding tracks in left side
Parts:
- added H6, H7, H8: MountingHole_Pad, winkeebs:HOLE_M2_TH, symbol Mechanical:MountingHole
- H1, H2, H3, H4, H5: footprint winkeebs:HOLE_M2 -> winkeebs:HOLE_M2_TH
Connections:
- net GND: now also TRRS1.1 (SLEEVE); no longer TRRS1.4 (RING2)
- net VCC: now also TRRS1.2 (TIP); no longer TRRS1.1 (SLEEVE)
- net at TRRS1.3 (RING1): no longer ESD1.1 (IO1)
- new net: ESD1.1 (IO1), TRRS1.4 (RING2)
- no-connect marks 15 -> 16
Other:
- moved on the sheet: ESD1, H1, H2, H3, H4, H5, Reset1, TRRS1
