File: pcb/right/Win-split-right.kicad_sch (KiCad schematic)
At the start: 172 parts, among them J2 Conn_01x04_Socket, U1 RP2040_ProMicro, U2 74AHCT1G125

Commit message: kicad 7
Parts:
- D1, D10, D11, D12, D13, D14, D15, D16, D17, D18, D19, D2, D20, D21, D22, D23, D24, D25, D26, D27, D28, D29, D3, D30, D31, D32, D33, D34, D35, D36, D37, D38, D39, D4, D5, D6, D7, D8, D9: footprint ScottoKeebs_Components:Diode_SOD-123 -> winkeebs:Diode_SOD-123
- LED1, LED17, LED18, LED19, LED2, LED20, LED21, LED22, LED3, LED32, LED33, LED34, LED35, LED36, LED37, LED38, LED39, LED4, LED5, LED6, LED7: footprint winkeebs:LED_MX_6028R-ROT -> PCM_marbastlib-mx:LED_MX_6028R-ROT
- LED10, LED11, LED12, LED13, LED14, LED15, LED25, LED26, LED27, LED28, LED29, LED9: footprint winkeebs:LED_MX_6028R -> PCM_marbastlib-mx:LED_MX_6028R
- LED16, LED30, LED31: footprint winkeebs:LED_MX_6028R-ROT -> PCM_marbastlib-mx:LED_MX_6028R
- LED23, LED24, LED8: footprint winkeebs:LED_MX_6028R -> PCM_marbastlib-mx:LED_MX_6028R-ROT
- MX1, MX10, MX11, MX12, MX13, MX14, MX15, MX16, MX17, MX18, MX19, MX2, MX20, MX21, MX22, MX25, MX26, MX27, MX28, MX29, MX3, MX30, MX31, MX32, MX33, MX37, MX38, MX39, MX4, MX5, MX6, MX7, MX9: footprint PCM_marbastlib-mx:SW_MX_HS_CPG151101S11_1u -> winkeebs:SW_MX_HS_CPG151101S11_1u
- MX23, MX34, MX35, MX36: footprint PCM_marbastlib-mx:SW_MX_HS_CPG151101S11_1u -> winkeebs:SW_MX_HS_CPG151101S11_1.25u
- MX24, MX8: footprint PCM_marbastlib-mx:SW_MX_HS_CPG151101S11_1u -> winkeebs:SW_MX_HS_CPG151101S11_1.5u
- renumbered H6 to H1, H7 to H2, H8 to H3, H9 to H4, H10 to H5

Commit message: prerouting right side
Parts:
- removed J2: Conn_01x04_Socket, Connector_PinHeader_2.54mm:PinHeader_1x04_P2.54mm_Vertical, symbol Connector:Conn_01x04_Socket
- removed OLED2: OLED_128x32, ScottoKeebs_Components:OLED_128x32, symbol ScottoKeebs:OLED_128x32
- added H6, H7, H8: MountingHole_Pad, winkeebs:HOLE_M2, symbol Mechanical:MountingHole
- added J1: Conn_01x04_Socket, Connector_PinHeader_2.54mm:PinHeader_1x04_P2.54mm_Vertical, symbol Connector:Conn_01x04_Socket
- added OLED1: OLED_128x32, ScottoKeebs_Components:OLED_128x32, symbol ScottoKeebs:OLED_128x32
- Reset1: LCSC (none) -> C231329
Connections:
- net GND: now also TRRS1.1 (SLEEVE), J1.1 (Pin_1), OLED1.1 (GND); no longer TRRS1.4 (RING2)
- net SCL: now also J1.3 (Pin_3), OLED1.3 (SCL)
- net SDA: now also J1.4 (Pin_4), OLED1.4 (SDA)
- net VCC: now also TRRS1.2 (TIP), J1.2 (Pin_2), OLED1.2 (VCC); no longer TRRS1.1 (SLEEVE)
- net at TRRS1.3 (RING1): no longer ESD1.1 (IO1)
- new net: ESD1.1 (IO1), TRRS1.4 (RING2)
Other:
- note added: "Left OLED and pin header"
- note added: "Left Reset switch"
- note added: "Left TRRS data connection"
- note removed: "Right OLED and pin header"
- note removed: "Right Reset switch"
- note removed: "Right TRRS data connection"
