File: pcb/right/_autosave-Win-split-right.kicad_pcb (KiCad board)
At the start: 2 copper layers, 213.2 x 120.4 mm, 175 parts, among them J2 Conn_01x04_Socket, U1 RP2040_ProMicro, U2 74AHCT1G125

Commit message: before rounding tracks in left side
Routing:
- net DATA: track 0.00 -> 31.6 mm, vias 0 -> 2
- net GND: track 0.00 -> 30.4 mm, vias 0 -> 1
- net Net-(ESD1-IO1): track 0.00 -> 28.2 mm, vias 0 -> 2
- net RESET: track 0.00 -> 12.8 mm
- net VCC: track 0.00 -> 9.62 mm, vias 0 -> 1
Changed lines of the file:
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@@
   (gr_circle (center 257.769737 52.703444) (end 259.919735 52.703444)
     (stroke (width 0.1) (type dot)) (fill none) (layer "Margin"))
+  (segment (start 84.031434 29.483308) (end 84.031434 23.520399) (width 0.25) (layer "F.Cu") (net 1))
+  (segment (start 82.119223 30.248111) (end 83.266631 30.248111) (width 0.25) (layer "F.Cu") (net 1))
+  (segment (start 79.061635 33.853107) (end 79.061635 33.305699) (width 0.25) (layer "F.Cu") (net 1))
+  (segment (start 83.266631 30.248111) (end 84.031434 29.483308) (width 0.25) (layer "F.Cu") (net 1))
+  (segment (start 79.061635 33.305699) (end 82.119223 30.248111) (width 0.25) (layer "F.Cu") (net 1))
+  (via (at 84.031434 23.520399) (size 0.6096) (drill 0.3048) (layers "F.Cu" "B.Cu") (net 1))
+  (via (at 79.061635 33.853107) (size 0.6096) (drill 0.3048) (layers "F.Cu" "B.Cu") (net 1))
+  (segment (start 86.238722 21.313111) (end 97.866635 21.313111) (width 0.25) (layer "B.Cu") (net 1))
+  (segment (start 75.983234 35.562759) (end 77.692886 33.853107) (width 0.25) (layer "B.Cu") (net 1))
+  (segment (start 77.692886 33.853107) (end 79.061635 33.853107) (width 0.25) (layer "B.Cu") (net 1))
+  (segment (start 84.031434 23.520399) (end 86.238722 21.313111) (width 0.25) (layer "B.Cu") (net 1))
+  (segment (start 77.502885 37.065361) (end 77.502885 32.324449) (width 0.25) (layer "F.Cu") (net 4))
+  (segment (start 82.626635 27.200699) (end 82.626635 26.393111) (width 0.25) (layer "F.Cu") (net 4))
+  (segment (start 77.502885 32.324449) (end 82.626635 27.200699) (width 0.25) (layer "F.Cu") (net 4))
   (segment (start 117.276635 21.948111) (end 117.276635 22.418112) (width 0.25) (layer "B.Cu") (net 6))
   (segment (start 117.276635 22.418112) (end 119.561635 24.703112) (width 0.25) (layer "B.Cu") (net 6))
@@
   (segment (start 143.470384 95.671611) (end 143.470384 96.141612) (width 0.25) (layer "B.Cu") (net 44))
   (segment (start 143.470384 96.141612) (end 145.755384 98.426612) (width 0.25) (layer "B.Cu") (net 44))
+  (segment (start 74.102885 31.424361) (end 73.481635 30.803111) (width 0.4) (layer "F.Cu") (net 70))
+  (segment (start 80.076635 21.303111) (end 82.626635 23.853111) (width 0.4) (layer "F.Cu") (net 70))
+  (segment (start 77.584579 21.303111) (end 80.076635 21.303111) (width 0.4) (layer "F.Cu") (net 70))
+  (segment (start 73.481635 30.803111) (end 73.481635 25.406055) (width 0.4) (layer "F.Cu") (net 70))
+  (segment (start 74.102885 37.065361) (end 74.102885 31.424361) (width 0.4) (layer "F.Cu") (net 70))
+  (segment (start 73.481635 25.406055) (end 77.584579 21.303111) (width 0.4) (layer "F.Cu") (net 70))
+  (segment (start 74.102885 39.615956) (end 74.940036 40.453107) (width 0.4) (layer "F.Cu") (net 70))
+  (segment (start 74.102885 37.065361) (end 74.102885 39.615956) (width 0.4) (layer "F.Cu") (net 70))
+  (via (at 74.940036 40.453107) (size 0.7) (drill 0.3048) (layers "F.Cu" "B.Cu") (net 70))
+  (segment (start 74.670156 38.21934) (end 74.670156 40.183227) (width 0.4) (layer "B.Cu") (net 70))
+  (segment (start 74.670156 40.183227) (end 74.940036 40.453107) (width 0.4) (layer "B.Cu") (net 70))
+  (segment (start 74.993285 37.896211) (end 74.670156 38.21934) (width 0.4) (layer "B.Cu") (net 70))
+  (segment (start 75.061635 34.453107) (end 75.061635 32.723111) (width 0.4) (layer "F.Cu") (net 78))
+  (segment (start 75.061635 32.723111) (end 78.081635 29.703111) (width 0.4) (layer "F.Cu") (net 78))
+  (via (at 75.061635 34.453107) (size 0.7) (drill 0.3048) (layers "F.Cu" "B.Cu") (net 78))
+  (segment (start 75.528546 36.557639) (end 74.988354 36.017447) (width 0.4) (layer "B.Cu") (net 78))
+  (segment (start 74.988354 34.526388) (end 75.061635 34.453107) (width 0.4) (layer "B.Cu") (net 78))
+  (segment (start 76.331857 36.557639) (end 75.528546 36.557639) (width 0.4) (layer "B.Cu") (net 78))
+  (segment (start 76.654985 36.234511) (end 76.331857 36.557639) (width 0.4) (layer "B.Cu") (net 78))
+  (segment (start 74.988354 36.017447) (end 74.988354 34.526388) (width 0.4) (layer "B.Cu") (net 78))
+  (segment (start 72.356635 39.148107) (end 72.356635 24.958107) (width 0.25) (layer "F.Cu") (net 86))
+  (segment (start 72.356635 24.958107) (end 73.661635 23.653107) (width 0.25) (layer "F.Cu") (net 86))
+  (segment (start 75.061635 41.853107) (end 72.356635 39.148107) (width 0.25) (layer "F.Cu") (net 86))
+  (via (at 73.661635 23.653107) (size 0.6096) (drill 0.3048) (layers "F.Cu" "B.Cu") (net 86))
+  (via (at 75.061635 41.853107) (size 0.6096) (drill 0.3048) (layers "F.Cu" "B.Cu") (net 86))
+  (segment (start 75.665036 38.567963) (end 75.665036 41.249706) (width 0.25) (layer "B.Cu") (net 86))
+  (segment (start 73.661635 23.653107) (end 74.611631 22.703111) (width 0.25) (layer "B.Cu") (net 86))
+  (segment (start 74.611631 22.703111) (end 78.081635 22.703111) (width 0.25) (layer "B.Cu") (net 86))
+  (segment (start 75.665036 41.249706) (end 75.061635 41.853107) (width 0.25) (layer "B.Cu") (net 86))
   (group "" (id fa6f942c-9fe1-47cb-b306-3a0bbb0b0c81)
     (members
