File: pcb/right/Win-split-right.kicad_pcb (KiCad board)
At the start: 2 copper layers, 4.1 x 3.8 mm, 131 parts, among them J2 Conn_01x04_Socket, U2 RP2040_ProMicro

Commit message: kicad 7
Parts:
- removed ESD2: SRV05-4, PCM_marbastlib-various:SOT-23-6-routable
- removed H10, H6, H7, H8, H9: MountingHole_Pad, winkeebs:HOLE_M2
- removed Reset2: Switch, Button_Switch_SMD:SW_SPST_B3U-1000P
- removed TRRS2: TRRS, ScottoKeebs_Components:TRRS_PJ-320A
- added C1: 100nF, Capacitor_SMD:C_0402_1005Metric, B.Cu at (116.4, 32.9)
- added C10: 100nF, Capacitor_SMD:C_0402_1005Metric, B.Cu at (135.4, 49.4)
- added C100: 100nF, Capacitor_SMD:C_0402_1005Metric, B.Cu at (101.3, 23.7)
- added C11: 100nF, Capacitor_SMD:C_0402_1005Metric, B.Cu at (154.5, 47.1)
- added C12: 100nF, Capacitor_SMD:C_0402_1005Metric, B.Cu at (173.5, 49.4)
- added C13: 100nF, Capacitor_SMD:C_0402_1005Metric, B.Cu at (193.0, 53.7)
- added C14: 100nF, Capacitor_SMD:C_0402_1005Metric, B.Cu at (211.5, 58.3)
- added C15: 100nF, Capacitor_SMD:C_0402_1005Metric, B.Cu at (230.0, 62.9)
- added C16: 100nF, Capacitor_SMD:C_0402_1005Metric, B.Cu at (276.2, 54.8)
- added C17: 100nF, Capacitor_SMD:C_0402_1005Metric, B.Cu at (116.4, 71.0)
- added C18: 100nF, Capacitor_SMD:C_0402_1005Metric, B.Cu at (135.4, 68.5)
- added C19: 100nF, Capacitor_SMD:C_0402_1005Metric, B.Cu at (154.5, 66.2)
- added C2: 100nF, Capacitor_SMD:C_0402_1005Metric, B.Cu at (135.4, 30.4)
- added C20: 100nF, Capacitor_SMD:C_0402_1005Metric, B.Cu at (173.5, 68.5)
- added C21: 100nF, Capacitor_SMD:C_0402_1005Metric, B.Cu at (193.0, 73.3)
- added C22: 100nF, Capacitor_SMD:C_0402_1005Metric, B.Cu at (211.5, 77.9)
- added C23: 100nF, Capacitor_SMD:C_0402_1005Metric, B.Cu at (241.6, 85.4)
- added C24: 100nF, Capacitor_SMD:C_0402_1005Metric, B.Cu at (253.1, 68.7)
- added C25: 100nF, Capacitor_SMD:C_0402_1005Metric, B.Cu at (116.4, 90.0)
- added C26: 100nF, Capacitor_SMD:C_0402_1005Metric, B.Cu at (135.4, 87.5)
- added C27: 100nF, Capacitor_SMD:C_0402_1005Metric, B.Cu at (154.5, 85.2)
- added C28: 100nF, Capacitor_SMD:C_0402_1005Metric, B.Cu at (173.5, 87.5)
- added C29: 100nF, Capacitor_SMD:C_0402_1005Metric, B.Cu at (193.1, 93.0)
- added C3: 100nF, Capacitor_SMD:C_0402_1005Metric, B.Cu at (154.5, 28.1)
- added C30: 100nF, Capacitor_SMD:C_0402_1005Metric, B.Cu at (218.5, 99.3)
- added C31: 100nF, Capacitor_SMD:C_0402_1005Metric, B.Cu at (243.9, 105.6)
- added C32: 100nF, Capacitor_SMD:C_0402_1005Metric, B.Cu at (97.3, 90.0)
- added C33: 100nF, Capacitor_SMD:C_0402_1005Metric, B.Cu at (109.2, 109.1)
- added C34: 100nF, Capacitor_SMD:C_0402_1005Metric, B.Cu at (142.6, 106.6)
- added C35: 100nF, Capacitor_SMD:C_0402_1005Metric, B.Cu at (166.4, 106.6)
- added C36: 100nF, Capacitor_SMD:C_0402_1005Metric, B.Cu at (200.0, 114.3)
- added C37: 100nF, Capacitor_SMD:C_0402_1005Metric, B.Cu at (220.8, 119.5)
- added C38: 100nF, Capacitor_SMD:C_0402_1005Metric, B.Cu at (239.3, 124.1)
- added C39: 100nF, Capacitor_SMD:C_0402_1005Metric, B.Cu at (257.8, 128.7)
- added C4: 100nF, Capacitor_SMD:C_0402_1005Metric, B.Cu at (173.5, 30.4)
- added C5: 100nF, Capacitor_SMD:C_0402_1005Metric, B.Cu at (193.0, 34.0)
- added C6: 100nF, Capacitor_SMD:C_0402_1005Metric, B.Cu at (211.5, 38.7)
- added C7: 100nF, Capacitor_SMD:C_0402_1005Metric, B.Cu at (230.0, 43.3)
- added C8: 100nF, Capacitor_SMD:C_0402_1005Metric, B.Cu at (253.1, 49.0)
- added C9: 100nF, Capacitor_SMD:C_0402_1005Metric, B.Cu at (116.4, 51.9)
- added ESD1: SRV05-4, PCM_marbastlib-various:SOT-23-6-routable, F.Cu at (75.8, 37.1)
- added H1: MountingHole_Pad, winkeebs:HOLE_M2, F.Cu at (104.0, 36.6)
- added H2: MountingHole_Pad, winkeebs:HOLE_M2, F.Cu at (23.9, 16.1)
- added H3: MountingHole_Pad, winkeebs:HOLE_M2, F.Cu at (23.9, 19.3)
- added H4: MountingHole_Pad, winkeebs:HOLE_M2, F.Cu at (23.9, 22.5)
- added H5: MountingHole_Pad, winkeebs:HOLE_M2, F.Cu at (23.9, 25.7)
- added Reset1: Switch, Button_Switch_SMD:SW_SPST_B3U-1000P, F.Cu at (75.8, 44.0)
- added TRRS1: TRRS, ScottoKeebs_Components:TRRS_PJ-320A, F.Cu at (75.8, 19.5)
- added U1: RP2040_ProMicro, winkeebs:RP2040_ProMicro_USBdn, F.Cu at (90.2, 35.3)
- D1, D10, D11, D12, D13, D14, D15, D16, D17, D18, D19, D2, D20, D21, D22, D23, D24, D25, D26, D27, D28, D29, D3, D30, D31, D32, D33, D34, D35, D36, D37, D38, D39, D4, D5, D6, D7, D8, D9: footprint ScottoKeebs_Components:Diode_SOD-123 -> winkeebs:Diode_SOD-123
- LED1, LED17, LED18, LED19, LED2, LED20, LED21, LED22, LED3, LED32, LED33, LED34, LED35, LED36, LED37, LED38, LED39, LED4, LED5, LED6, LED7: footprint winkeebs:LED_MX_6028R-ROT -> PCM_marbastlib-mx:LED_MX_6028R-ROT
- LED10, LED11, LED12, LED13, LED14, LED15, LED25, LED26, LED27, LED28, LED29, LED9: footprint winkeebs:LED_MX_6028R -> PCM_marbastlib-mx:LED_MX_6028R
- LED16, LED30, LED31: footprint winkeebs:LED_MX_6028R-ROT -> PCM_marbastlib-mx:LED_MX_6028R
- LED23, LED24, LED8: footprint winkeebs:LED_MX_6028R -> PCM_marbastlib-mx:LED_MX_6028R-ROT
- MX1, MX10, MX11, MX12, MX13, MX14, MX15, MX16, MX17, MX18, MX19, MX2, MX20, MX21, MX22, MX25, MX26, MX27, MX28, MX29, MX3, MX31, MX32, MX37, MX38, MX39, MX4, MX5, MX6, MX7, MX9: footprint ScottoKeebs_Hotswap:Hotswap_MX_Plated_1.00u -> winkeebs:SW_MX_HS_CPG151101S11_1u; moved to B.Cu
- MX23: footprint ScottoKeebs_Hotswap:Hotswap_MX_Plated_2.25u -> winkeebs:SW_MX_HS_CPG151101S11_1.25u; moved to B.Cu
- MX24: footprint ScottoKeebs_Hotswap:Hotswap_MX_Plated_1.00u -> winkeebs:SW_MX_HS_CPG151101S11_1.5u; moved to B.Cu
- MX30: footprint ScottoKeebs_Hotswap:Hotswap_MX_Plated_1.75u -> winkeebs:SW_MX_HS_CPG151101S11_1u; moved to B.Cu
- MX33: footprint ScottoKeebs_Hotswap:Hotswap_MX_Plated_2.25u -> winkeebs:SW_MX_HS_CPG151101S11_1u; moved to B.Cu
- MX34, MX35, MX36: footprint ScottoKeebs_Hotswap:Hotswap_MX_1.25u -> winkeebs:SW_MX_HS_CPG151101S11_1.25u; moved to B.Cu
- MX8: footprint ScottoKeebs_Hotswap:Hotswap_MX_Plated_1.50u -> winkeebs:SW_MX_HS_CPG151101S11_1.5u; moved to B.Cu
- U2: value RP2040_ProMicro -> 74AHCT1G125; footprint winkeebs:RP2040_ProMicro_USBdn -> Package_TO_SOT_SMD:SOT-23-5; moved to B.Cu
- moved D25 197.7 mm to (119.6, 83.5)
- moved D11 197.7 mm to (157.7, 40.6)
- moved D32 197.7 mm to (100.5, 83.5)
- moved D17 197.7 mm to (119.6, 64.5)
- moved D26 197.7 mm to (138.6, 81.0)
- moved D9 197.7 mm to (119.6, 45.4)
- moved D28 197.7 mm to (176.7, 81.0)
- moved D3 197.7 mm to (157.7, 21.6)
- moved D18 197.7 mm to (138.6, 62.0)
- moved D12 197.7 mm to (176.7, 42.9)
- moved D34 197.7 mm to (145.8, 100.1)
- moved D1 197.7 mm to (119.6, 26.4)
- moved D2 197.7 mm to (138.6, 23.9)
- moved D19 197.7 mm to (157.7, 59.7)
- moved D35 197.7 mm to (169.6, 100.1)
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Connections:
- LED1 pad 3: LED -> LED_5v
- U2 pad 1: LED -> GND
- U2 pad 2: SDA -> LED_3v3
- U2 pad 3: SCL -> GND
- U2 pad 4: ROW0 -> LED_5v
- U2 pad 5: ROW1 -> +5V
Routing:
- net Net-(D31-A): track 4.84 -> 3.70 mm
- net Net-(D7-A): track 4.84 -> 3.70 mm
- net Net-(D23-A): track 4.84 -> 3.70 mm
- net Net-(D38-A): track 4.84 -> 3.70 mm
- net Net-(D16-A): track 4.84 -> 3.70 mm
- net Net-(D21-A): track 4.84 -> 3.70 mm
- net Net-(D22-A): track 4.84 -> 3.70 mm
- net Net-(D8-A): track 4.84 -> 3.70 mm
- net Net-(D10-A): track 4.84 -> 3.70 mm
- net Net-(D37-A): track 4.84 -> 3.70 mm
- net Net-(D15-A): track 4.84 -> 3.70 mm
- net Net-(D13-A): track 4.84 -> 3.70 mm
- net Net-(D14-A): track 4.84 -> 3.70 mm
- net Net-(D39-A): track 4.84 -> 3.70 mm
- net Net-(D17-A): track 4.84 -> 3.70 mm
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
Commit message: prerouting right side
Parts:
- removed J2: Conn_01x04_Socket, Connector_PinHeader_2.54mm:PinHeader_1x04_P2.54mm_Vertical
- removed OLED2: OLED_128x32, ScottoKeebs_Components:OLED_128x32
- added H6: MountingHole_Pad, winkeebs:HOLE_M2, F.Cu at (177.1, 92.1)
- added H7: MountingHole_Pad, winkeebs:HOLE_M2, F.Cu at (120.7, 73.4)
- added H8: MountingHole_Pad, winkeebs:HOLE_M2, F.Cu at (77.8, 84.2)
- added J1: Conn_01x04_Socket, Connector_PinHeader_2.54mm:PinHeader_1x04_P2.54mm_Vertical, F.Cu at (86.4, 55.6)
- ESD1, R3: moved to B.Cu
- moved H4 237.4 mm to (244.7, 109.7)
- moved H3 236.3 mm to (257.8, 52.7)
- moved H5 180.3 mm to (200.9, 59.5)
- moved H2 157.5 mm to (180.2, 35.7)
- moved C100 12.2 mm to (90.8, 29.9)
- moved U2 12.2 mm to (90.8, 27.1)
- moved Reset1 6.94 mm to (75.8, 37.1)
- moved D17 2.81 mm to (120.1, 61.7), turned to -90 degrees
- moved D11 2.81 mm to (158.2, 37.9), turned to -90 degrees
- moved D20 2.81 mm to (177.2, 59.2), turned to -90 degrees
- moved D27 2.81 mm to (158.2, 76.0), turned to -90 degrees
- moved D34 2.81 mm to (146.3, 97.3), turned to -90 degrees
- moved D35 2.81 mm to (170.1, 97.3), turned to -90 degrees
- moved D25 2.81 mm to (120.1, 80.7), turned to -90 degrees
- moved D32 2.81 mm to (101.0, 80.7), turned to -90 degrees
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Connections:
- TRRS1 pad 1: VCC -> GND
- TRRS1 pad 2: unconnected-(TRRS1-TIP-Pad2) -> VCC
- TRRS1 pad 3: Net-(ESD1-IO1) -> unconnected-(TRRS1-RING1-Pad3)
- TRRS1 pad 4: GND -> Net-(ESD1-IO1)
Routing:
- net Net-(D32-A): track 3.70 -> 0.00 mm
- net Net-(D25-A): track 3.70 -> 0.00 mm
- net Net-(D34-A): track 3.70 -> 0.00 mm
- net Net-(D9-A): track 3.70 -> 0.00 mm
- net Net-(D20-A): track 3.70 -> 0.00 mm
- net Net-(D19-A): track 3.70 -> 0.00 mm
- net Net-(D18-A): track 3.70 -> 0.00 mm
- net Net-(D10-A): track 3.70 -> 0.00 mm
- net Net-(D4-A): track 3.70 -> 0.00 mm
- net Net-(D3-A): track 3.70 -> 0.00 mm
- net Net-(D2-A): track 3.70 -> 0.00 mm
- net Net-(D1-A): track 3.70 -> 0.00 mm
- net Net-(D17-A): track 3.70 -> 0.00 mm
- net Net-(D12-A): track 3.70 -> 0.00 mm
- net Net-(D11-A): track 3.70 -> 0.00 mm
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Other:
- board size 4.1 x 3.8 mm -> 213.2 x 120.4 mm
